File: 17.kicad_sch (KiCad schematic)
At the start: 59 parts, among them J21 CON_RJ45-28_LPJG17512AONL, Q14 BSS138LT1G, Q16 BSS138LT1G, Q21 BSS138LT1G, U27 TMUX154EDGSR, U31 SN74LVC1G08DBVRE4, U80 DP83869HMRGZT

Commit message: fix joint, offpage, and typo
DRC errors are cleared, some warnings remain.
Parts:
- removed *: MISTRAL_TITLEBLK_CSIZE, symbol 17-altium-import:root_0_MISTRAL_TITLEBLK_CSIZE
Connections:
- net DGND: now also C101.2, C106.2, C110.2, C111.2, C112.2, C114.2, C124.2, C385.2, C389.2, C392.2, C394.2, C395.2, C401.2, C99.2, R135.2, R359.2, R363.2, R371.2, R385.2, R386.2, R563.2
- net GPIO_RGMII2_RST: now also R380.1
- net PRG1_ETH2_GPIO_1: now also R340.2, R341.1
- net PRG1_ETH2_LED2: now also R616.1
- net PRG1_ETH2_LED3: now also R615.1
- net PRG1_ETH2_LED_1000/RX_ER: now also R386.1, R388.2
- net PRG1_ETH2_LED_ACT: now also R385.1, R387.2
- net PRG1_ETH2_LED_LINK: now also R562.2, R563.1
- net PRG1_RGMII2_RD0: now also R126.2, R359.1
- net PRG1_RGMII2_RD1: now also R128.2, R363.1
- net PRG1_RGMII2_RESETn: now also R367.1
- net PRG1_RGMII2_RX_CTL: now also R135.1, R366.2
- net PRG_EARTH: now also J21.SH4
- net VCC_3V3_SYS: now also C101.1, C128.1, C385.1, C389.1, C89.1, C99.1, R128.1, R340.1, R366.1, R369.1, R387.1, R388.1, R562.1
- net VDD_1V1: now also C105.1, C110.1, C112.1, C124.1, C395.1, C401.1, U80.39 (VDD1P1), U80.6 (VDDA1P1)
- net VDD_2V5: now also C106.1, C111.1, C114.1, C392.1, U80.3 (VDDA2P5)
- net at TP69.1 (TP), U80.48 (VDDA1P8_2): now also U80.13 (VDDA1P8_1)
- no-connect marks 10 -> 8
Other:
- moved on the sheet: R615, R616
