File: 18.kicad_sch (KiCad schematic)
At the start: 57 parts, among them J21 CON_RJ45-28_LPJG17512AONL, Q15 BSS138LT1G, Q20 BSS138LT1G, Q4 BSS138LT1G, U19 SN74LVC1G08DBVRE4, U20 DP83869HMRGZT

Commit message: fix joint, offpage, and typo
DRC errors are cleared, some warnings remain.
Parts:
- removed *: MISTRAL_TITLEBLK_CSIZE, symbol 18-altium-import:root_0_MISTRAL_TITLEBLK_CSIZE
Connections:
- net DGND: now also C293.2, C297.2, C301.2, C305.2, C306.2, C313.2, C320.2, C349.2, C369.2, C68.2, C73.2, C76.2, C78.2, C83.2, R100.2, R107.2, R108.2, R301.2, R304.2, R565.2, R96.2, R97.2
- net GPIO_RGMII1_RST: now also R300.1
- net PRG1_ETH3_GPIO_1: now also R114.2, R115.1
- net PRG1_ETH3_LED2: now also R613.1
- net PRG1_ETH3_LED3: now also R612.1
- net PRG1_ETH3_LED_1000/RX_ER: now also R94.2, R96.1
- net PRG1_ETH3_LED_ACT: now also R95.2, R97.1
- net PRG1_ETH3_LED_LINK: now also R564.2, R565.1
- net PRG1_RGMII1_RD0: now also R108.1, R310.2
- net PRG1_RGMII1_RD1: now also R107.1, R308.2
- net PRG1_RGMII1_RESETn: now also R102.1
- net PRG1_RGMII1_RX_CTL: now also R100.1, R101.2
- net PRG_EARTH: now also J21.SH2, R304.1
- net VCC_3V3_SYS: now also C320.1, C349.1, C369.1, C67.1, C83.1, R101.1, R103.2, R104.1, R114.1, R308.1, R564.1, R94.1, R95.1, U20.18 (VDDIO)
- net VDD_1V1: now also C293.1, C301.1, C306.1, C316.1, C68.1, C78.1, U20.39 (VDD1P1), U20.6 (VDDA1P1)
- net VDD_2V5: now also C297.1, C305.1, C313.1, C73.1
- net at TP19.1 (TP), U20.48 (VDDA1P8_2): now also U20.13 (VDDA1P8_1)
- no-connect marks 10 -> 8
