File: 22.kicad_sch (KiCad schematic)
At the start: 57 parts, among them J28 CON_MUSB-B_5_F, U58 TPD4E004DRYR, U59 TM4C1294NCPDTT3R, U61 TPS79601DRBR, U95 LM4040B25IDCKR, Y2 16.000MHZ

Commit message: fix joint, offpage, and typo
DRC errors are cleared, some warnings remain.
Parts:
- removed *: MISTRAL_TITLEBLK_CSIZE, symbol 22-altium-import:root_0_MISTRAL_TITLEBLK_CSIZE
Connections:
- net DGND: now also C166.2, C175.2, C176.2, C180.2, C185.1, C186.2, C191.2, C192.1, C196.1, C453.1, R207.1, R208.1, R209.1, U59.114 (GND), U59.17 (GND), U59.48 (GND), U59.58 (GND), U59.66 (XOSC0), U59.80 (GND), U61.6 (GND), U61.9 (PAD), U95.1 (ANODE)
- net VCC3V3_XDS: now also C166.1, C175.1, C176.1, C191.1, C192.2, C196.2, C198.1, R203.1, R204.1, R558.2, R559.2, R560.2, U59.101 (VDD), U59.113 (VDD), U59.122 (VDD), U59.16 (VDD), U59.26 (VDD), U59.28 (VDD), U59.39 (VDD), U59.47 (VDD), U59.51 (VDD), U59.52 (VDD), U59.69 (VDD), U59.7 (VDD), U59.79 (VDD), U59.8 (VDDA), U59.90 (VDD), U61.3 (OUT1), U61.4 (OUT2)
- net VDDC_1V2: now also U59.115 (VDDC)
- net VREF: now also U95.3 (CATHODE)
- net XDS_RSTn: now also R199.1
- net XDS_SHIELD: now also J28.SH1, J28.SH2, J28.SH4, J28.SH5
- net XDS_USB_VBUS: now also U61.1 (IN1), U61.2 (IN2), U61.8 (EN)
- net at C198.2, U61.5 (NR/FB): now also R204.2, R561.1
- net at R200.1: now also C193.2, U59.68 (VBAT)
- net at C447.2: now also R467.2, U59.96 (PB1/USB0VBUS)
- net at R468.1, R469.2: now also U59.1 (PD0/AIN15)
- net at R207.2, R559.1: now also U59.61 (PK6)
- net at R206.2, R560.1: now also U59.60 (PK7)
- net at R209.2, R557.1: now also U59.63 (PK4)
- net at U59.62 (PK5): now also R208.2, R558.1
- no-connect marks 82 -> 79
