File: 26.kicad_sch (KiCad schematic)
At the start: 57 parts, among them J26 CON_MUSB-B_5_F, U42 TPD4E004DRYR, U43 TPS73533DRVR, U82 SN74AVC4T245RSVR, U84 SN74AVC4T245RSVR, U87 FT4232HL, U89 SN74AVC4T245RSVR, U92 93LC46B, Y3 12.000MHz

Commit message: fix joint, offpage, and typo
DRC errors are cleared, some warnings remain.
Parts:
- removed *: MISTRAL_TITLEBLK_CSIZE, symbol 26-altium-import:root_0_MISTRAL_TITLEBLK_CSIZE
Connections:
- net DGND: now also C154.1, C158.2, C160.1, C412.1, C413.1, C419.1, C420.1, C423.1, C442.1, D6.1, U43.7 (EP), U82.10 (GND1), U82.16 (~{2OE}), U84.10 (GND1), U84.16 (~{2OE}), U87.10 (AGND), U87.11 (GND3), U87.15 (GND4), U87.25 (GND5), U87.35 (GND6), U87.47 (GND7), U87.5 (GND2), U87.51 (GND8), U89.10 (GND1), U89.16 (~{2OE})
- net FT4232_USB_VBUS: now also C152.2, C154.2, D6.2, U43.6 (IN)
- net GNDUSB: now also C160.2, J26.SH1, J26.SH2, J26.SH4, J26.SH6
- net VCC_1V8_FT4232: now also C419.2, C420.2, C440.2, C441.1, U87.12 (VCORE), U87.37 (VCORE), U87.49 (VREGOUT), U87.64 (VCORE)
- net VCC_3V3_FT4232: now also C158.1, C413.2, C423.2, C445.2, R186.2, R191.2, U82.2 (VCCB), U84.2 (VCCB), U87.20 (VCCIO), U87.31 (VCCIO), U87.42 (VCCIO), U89.2 (VCCB)
- net VCC_3V3_SYS: now also U82.3 (VCCA), U84.3 (VCCA), U89.3 (VCCA)
- net VPHY_3V3_FT4232: now also FB24.1
- net VPLL_3V3_FT4232: now also FB23.1
- net at C439.1, U87.2 (OSCI): now also Y3.1
- net at Y3.2: now also C433.1, U87.3 (OSCO)
- no-connect marks 29 -> 27
Other:
- moved on the sheet: C416, D6
