File: 19.kicad_sch (KiCad schematic)
At the start: 27 parts, among them J38 CON_FLEX_40X1_FH12A-40S-0.5SH, U51 TCA9617BDGKR

Commit message: fix joint, offpage, and typo
DRC errors are cleared, some warnings remain.
Parts:
- removed *: MISTRAL_TITLEBLK_CSIZE, symbol 19-altium-import:root_0_MISTRAL_TITLEBLK_CSIZE
Connections:
- net BOOTMODE_I2C_SCL: now also R550.2
- net BOOTMODE_I2C_SDA: now also R551.2
- net DGND: now also C469.2, J38.16, J38.34, J38.41
- net TEST_GPIO3: now also R525.1
- net TEST_GPIO4: now also R526.1
- net VCC3V3_TA: now also C181.1, C469.1, C472.1, J38.1, J38.2, R494.1, R522.2, R523.2, R524.2, R525.2, R526.2, U51.1 (VCCA)
- net VCC_3V3_SYS: now also C161.1

Commit message: fixpcb.
TODO clean up zones and keepouts on all layers. (top done almost)
Connections:
- net VCC3V3_TA: now also R550.1, R551.1
Changed lines of the file:
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@@
+	)
+	(junction
+		(at 254 111.76)
+		(diameter 0)
+		(color 0 0 0 0)
 	)
 	(junction
@@
 	(wire
 		(pts
-			(xy 248.92 111.76) (xy 259.08 111.76)
+			(xy 248.92 111.76) (xy 254 111.76)
 		)
 		(stroke
@@
 		)
 		(stroke
+			(width 0)
+			(type default)
+		)
+	)
+	(wire
+		(pts
+			(xy 254 111.76) (xy 259.08 111.76)
+		)
+		(stroke
