File: 09.kicad_sch (KiCad schematic)
At the start: 62 parts, among them U23 AM6442BSFGHAALV

Commit message: fix joint, offpage, and typo
DRC errors are cleared, some warnings remain.
Parts:
- removed *: MISTRAL_TITLEBLK_CSIZE, symbol 09-altium-import:root_0_MISTRAL_TITLEBLK_CSIZE
Connections:
- net DGND: now also C289.2, C298.2, C322.2, C344.2, C347.2, C348.2, C350.2, C353.2, C355.2, C356.2, C357.2, C362.2, C373.2, C375.2, C380.2, C390.2, C396.2, C400.2, C92.2, C93.2
- net SOC_DVDD1V8: now also U23.M15 (VDDSHV4)
- net SoC_DVDD3V3: now also U23.G10 (VDDSHV_MCU), U23.G12 (VDDSHV0), U23.G14 (VDDSHV0), U23.G8 (VDDSHV_MCU), U23.M7 (VDDSHV1), U23.N6 (VDDSHV1), U23.P14 (VDDSHV3), U23.P15 (VDDSHV3), U23.P7 (VDDSHV1), U23.R10 (VDDSHV2), U23.R8 (VDDSHV2), U23.T9 (VDDSHV2)
- net VDDAR_0P85_SERDES0: now also C344.1, C356.1, C362.1, C92.1, C93.1, U23.P11 (VDDA_0P85_SERDES0_C), U23.P13 (VDDA_0P85_SERDES0)
- net VDDAR_0P85_USB0: now also C350.1
- net VDDAR_CORE: now also R75.1
- net VDDA_1V8_MCU: now also C353.1
- net VDDA_1V8_SERDES: now also C375.1
- net VDDA_1V8_USB0: now also C380.1
- net VDDA_CORE: now also R78.2
- net VDDA_PLL0: now also C355.1
- net VDDA_PLL1: now also C322.1
- net VDDA_PLL2: now also C347.1
- net VDDA_SYS_MON: now also R314.2, R315.1
- net VDDR_CORE: now also R106.2, U23.M13 (VDDR_CORE)
- net VDDSHV_SD_IO: now also U23.L15 (VDDSHV5)
- net VDDS_MMC0/ADC0_VREFP: now also R698.2, R699.1
- net VDD_CORE: now also R78.1, U23.J12 (VDD_CORE), U23.K11 (VDD_CORE), U23.K9 (VDD_CORE), U23.L12 (VDD_CORE), U23.L8 (VDD_CORE), U23.M11 (VDD_CORE), U23.M9 (VDD_CORE), U23.N10 (VDD_CORE), U23.N8 (VDD_CORE), U23.P9 (VDD_CORE)
- net VDD_DDR4: now also U23.G6 (VDDS_DDR), U23.H7 (VDDS_DDR), U23.J6 (VDDS_DDR), U23.K7 (VDDS_DDR), U23.L6 (VDDS_DDR)
- net VDD_DLL_MMC0: now also C373.1

Commit message: a lot, mpu power almost ready.
Parts:
- removed C103, C120, C299, C327, C341, C363, C377, C398, C74, C88: 4.7uF, CAP0402_0-75, symbol 09-altium-import:root_0_CAP_Dup1
- removed C121, C300, C340, C358, C365, C368, C387, C399, C75, C91, C92, C93: 0.1uF, CAP0201_0-5, symbol 09-altium-import:root_0_CAP_Dup3
- removed C289, C298, C348, C357, C390, C391, C396: 1uF, CAP0201_0-5, symbol 09-altium-import:root_0_CAP_Dup3
- removed C322, C344, C347, C350, C353, C355, C356, C362, C373, C375, C380: 0.01uF, CAP0402N, symbol 09-altium-import:root_0_CAP_Dup2
- removed C400: 3.3uF, CAP0603_1, symbol 09-altium-import:root_0_CAP_Dup3
- removed FB13, FB15, FB18, FB20, FB3, FB5, FB6: 120E, IND0603_1, symbol 09-altium-import:root_1_INDUCTOR_FERRITE
- removed FB16, FB17, FB4: 26E, IND0603_1, symbol 09-altium-import:root_1_INDUCTOR_FERRITE
- removed R106, R297, R75, R78: 0E, RES1210_0-75, symbol 09-altium-import:root_1_RESISTOR
- removed R698, R699: 0E, RES0201_0-5, symbol 09-altium-import:root_1_RESISTOR_Dup5
- added C103, C299, C327, C377, C74: 100n, Abacus:NFM15, symbol Device:Filter_EMI_C
- added C120, C341, C363, C398, C88: Filter_EMI_C, Abacus:NFM15, symbol Device:Filter_EMI_C
- added C289, C298, C348, C357, C390, C391, C396: 1u,20%,6.3V, Abacus:C_0201_0603Metric_0.64x0.32mm_Courtyard, symbol JLCE_C0201:1u,20%,6.3V
- added C344, C350, C356, C362, C368, C375, C380, C7: 100n,10%,10V, Abacus:C_0201_0603Metric_0.64x0.32mm_Courtyard, symbol JLCE_C0201:100n,10%,10V
- added C400: 3.3u, Capacitor_SMD:C_0402_1005Metric, symbol Abacus:C0402
Connections:
- net VDDA_CORE is gone; now on net VDD_CORE: U23.K13 (VDD_MMC0)
- net VDDR_CORE is gone; now on net VDD_CORE: U23.L10 (VDDR_CORE), U23.M13 (VDDR_CORE)
- net VDDS_MMC0/ADC0_VREFP is gone; now on net VDDA_ADC: U23.J15 (ADC0_REFP)
- net CAP_VDDS0: now also C390.1
- net CAP_VDDS1: now also C298.1
- net CAP_VDDS2: now also C348.1
- net CAP_VDDS3: now also C357.1
- net CAP_VDDS4: now also C396.1
- net CAP_VDDS5: now also C391.1
- net CAP_VDDS_MCU: now also C289.1
- net DGND: now also C289.2, C298.2, C344.2, C348.2, C350.2, C356.2, C357.2, C362.2, C368.2, C375.2, C380.2, C390.2, C391.2, C396.2, C400.2
- net VDDAR_0P85_SERDES0: now also C344.1, C356.1, C362.1, C88.3
- net VDDAR_0P85_USB0: now also C341.3, C350.1
- net VDDA_1V8: now also C103.1, C120.1, C299.1, C327.1, C363.1, C398.1, C74.1
- net VDDA_1V8_MCU: now also C103.3
- net VDDA_1V8_SERDES: now also C120.3, C375.1
- net VDDA_1V8_USB0: now also C380.1, C398.3
- net VDDA_ADC: now also C363.3, C368.1
- net VDDA_PLL0: now also C327.3
- net VDDA_PLL1: now also C299.3
- net VDDA_PLL2: now also C74.3
- net VDDSHV_SD_IO: now also C400.1
- net VDD_CORE: now also C341.1, C377.1, C88.1
- net VDD_DLL_MMC0: now also C377.3
- net VPP_1V8: now also C7.1
- net SOC_DVDD1V8 renamed VCC1V8
- net SoC_DVDD3V3 renamed VCC_3V3_SYS
- new net GND: C103.2, C120.2, C299.2, C327.2, C341.2, C363.2, C377.2, C398.2, C7.2, C74.2, C88.2
Other:
- note removed: "R1"
- note removed: "R2"
- note removed: "R3"
- note removed: "R4"
