File: 10.kicad_sch (KiCad schematic)
At the start: 79 parts

Commit message: fix joint, offpage, and typo
DRC errors are cleared, some warnings remain.
Parts:
- removed *: MISTRAL_TITLEBLK_CSIZE, symbol 10-altium-import:root_0_MISTRAL_TITLEBLK_CSIZE
Connections:
- net DGND: now also C278.2, C285.2, C290.2, C292.2, C294.2, C296.2, C302.2, C303.2, C304.2, C307.2, C308.2, C309.2, C310.2, C311.2, C312.2, C314.2, C315.2, C317.2, C318.2, C319.2, C321.2, C323.2, C324.2, C325.2, C326.2, C328.2, C329.2, C330.2, C331.2, C332.2, C333.2, C335.2, C336.2, C337.2, C338.2, C339.2, C342.2, C343.2, C345.2, C346.2, C352.2, C354.2, C359.2, C360.2, C361.2, C366.1, C370.2, C371.2, C372.2, C374.2, C376.2, C378.2, C379.2, C382.2, C383.2, C475.2, C483.2, C484.2, C98.1
- net SOC_DVDD1V8: now also C359.1, C371.1, C379.1, C383.1, C98.2
- net SoC_DVDD3V3: now also C304.1, C309.1, C312.1, C319.1, C321.1, C326.1, C328.1, C331.1, C333.1, C337.1, C343.1, C360.1, C361.1, C366.2, C374.1, C376.1, C378.1
- net VDDA_1V8: now also C338.1, C342.1, C346.1, C370.1
- net VDDR_CORE: now also C330.1, C475.1, R307.1, TP61.1 (TP)
- net VDDSHV_SD_IO: now also C372.1
- net VDD_CORE: now also C315.1, C318.1, C323.1, C324.1, C325.1, C329.1, C332.1, C335.1, C336.1, C339.1, C345.1, C352.1, C354.1, C483.1, C484.1, R298.1, TP55.1 (TP)
- net VDD_DDR4: now also C290.1, C294.1, C302.1, C303.1, C307.1, C308.1, C310.1, C311.1, C314.1, C317.1
- net VDD_MMC1: now also C382.1
- net at C279.1: now also C278.1, C285.1, R298.2
- net at C292.1: now also C291.1, C296.1, R307.2

Commit message: a lot, mpu power almost ready.
Parts:
- removed C278, C279, C285, C291, C292, C296: 0.1uF, CAP0402_0-75, symbol 10-altium-import:root_0_CAP_Dup3
- removed C294, C336: 1uF, CAP0402_0-75, symbol 10-altium-import:root_0_mirrored_CAP_Dup3
- removed C302, C303, C304, C307, C308, C309, C310, C311, C312, C314, C315, C317, C318, C319, C321, C323, C324, C325, C326, C328, C329, C330, C331, C332, C333, C337, C338, C339, C342, C343, C345, C346, C351, C352, C354, C359, C360, C361, C370, C371, C372, C374, C376, C378, C379, C381, C382, C383, C475, C483, C484: 0.1uF, CAP0201_0-5, symbol 10-altium-import:root_0_CAP_Dup3
- removed C334: 10uF, CAP0402_0-75, symbol 10-altium-import:root_0_CAP_Dup1
- removed C335, C79: 4.7uF, CAP0402_0-75, symbol 10-altium-import:root_0_CAP_Dup1
- removed R298, R307: 50E_0.1%, RES0402_0-5, symbol 10-altium-import:root_0_RESISTOR_Dup6
- removed TP54, TP55, TP61, TP63: THRU HOLE, TP_40X65, symbol 10-altium-import:root_2_mirrored_TESTPOINT
- added C294: 1u,20%,6.3V, Abacus:C_0201_0603Metric_0.64x0.32mm_Courtyard, symbol JLCE_C0201:1u,20%,6.3V
- added C302, C303, C304, C307, C309, C310, C311, C312, C314, C315, C317, C318, C319, C321, C323, C325, C326, C328, C329, C330, C331, C332, C333, C337, C338, C339, C342, C343, C345, C346, C351, C352, C354, C359, C360, C361, C370, C376, C379, C381, C382, C383, C4, C475, C483, C484: 100n,10%,10V, Abacus:C_0201_0603Metric_0.64x0.32mm_Courtyard, symbol JLCE_C0201:100n,10%,10V
- added C334, C335: 22u,±20%,6.3V, Abacus:C_0603_1608Metric_1.28x0.64mm_Courtyard, symbol JLC_C0603:22u,±20%,6.3V
- added C336: 10u,±10%,10V, Abacus:C_0603_1608Metric_1.28x0.64mm_Courtyard, symbol JLC_C0603:10u,±10%,10V
- added C37: 4.7u,20%,6.3V, Abacus:C_0201_0603Metric_0.64x0.32mm_Courtyard, symbol JLCE_C0201:4.7u,20%,6.3V
- added C79: 4.7u,20%,10V, Abacus:C_0402_1005Metric_for_0.25mm_grid, symbol JLC_C0402:4.7u,20%,10V
Connections:
- net VDDR_CORE is gone; now on net VDD_CORE: C86.2, C87.1
- net DGND: now also C294.2, C302.2, C303.2, C304.2, C307.2, C309.2, C310.2, C311.2, C312.2, C314.2, C315.2, C317.2, C318.2, C319.2, C321.2, C323.2, C325.2, C326.2, C328.2, C329.2, C330.2, C331.2, C332.2, C333.2, C334.2, C335.2, C336.2, C337.2, C338.2, C339.2, C342.2, C343.2, C345.2, C346.2, C351.2, C352.2, C354.2, C359.2, C360.2, C361.2, C37.2, C370.2, C376.2, C379.2, C381.2, C382.2, C383.2, C4.2, C475.2, C483.2, C484.2, C79.2
- net VDDA_1V8: now also C338.1, C342.1, C346.1, C370.1, C79.1
- net VDDSHV_SD_IO: now also C381.1
- net VDD_CORE: now also C315.1, C318.1, C323.1, C325.1, C329.1, C330.1, C332.1, C334.1, C335.1, C336.1, C339.1, C345.1, C352.1, C354.1, C37.1, C4.1, C475.1, C483.1, C484.1
- net VDD_DDR4: now also C294.1, C302.1, C303.1, C307.1, C310.1, C311.1, C314.1, C317.1
- net VDD_MMC1: now also C382.1
- net SOC_DVDD1V8 renamed VCC1V8
- net VCC1V8: now also C359.1, C379.1, C383.1
- net SoC_DVDD3V3 renamed VCC_3V3_SYS
- net VCC_3V3_SYS: now also C304.1, C309.1, C312.1, C319.1, C321.1, C326.1, C328.1, C331.1, C333.1, C337.1, C343.1, C351.1, C360.1, C361.1, C376.1
Other:
- note added: "VDDA for K13, VDD_MMC0"
- note removed: "Core & Array Core Supply Kelvin Sensing"
