File: 12.kicad_sch (KiCad schematic)
At the start: 75 parts, among them U13 MT40A1G16KD-062E IT:E, U23 AM6442BSFGHAALV

Commit message: fix joint, offpage, and typo
DRC errors are cleared, some warnings remain.
Parts:
- removed *: MISTRAL_TITLEBLK_CSIZE, symbol 12-altium-import:root_0_MISTRAL_TITLEBLK_CSIZE
Connections:
- net DDR_RESET#: now also R66.2, R67.1
- net DDR_TEN: now also R62.2, R63.1
- net DDR_VPP: now also C227.2, C270.2, U13.B1 (VPP)
- net DGND: now also C222.2, C223.2, C224.2, C227.1, C229.2, C232.2, C233.2, C236.2, C239.2, C241.2, C244.2, C246.2, C250.2, C251.2, C264.2, C267.2, C268.2, C270.1, C60.2, C61.2, C62.2, C63.2, U13.A2 (VSSQ), U13.A8 (VSSQ), U13.B2 (VSS), U13.C9 (VSSQ), U13.D2 (VSSQ), U13.D8 (VSSQ), U13.E1 (VSS), U13.E3 (VSSQ), U13.E8 (VSSQ), U13.E9 (VSS), U13.F1 (VSSQ), U13.G8 (VSS), U13.H1 (VSSQ), U13.K1 (VSS), U13.K9 (VSS), U13.M9 (VSS), U13.N1 (VSS), U13.T1 (VSS)
- net VDDR_VTT: now also C244.1, C246.1, C254.1, C58.1, C60.1, C61.1, C63.1, R264.2, R271.2, R273.2, R287.2, R288.2, R289.2, R291.2, R46.2, R77.2, R83.2, R84.2, R85.2, R86.2, R87.2, R88.2, R89.2, R90.2
- net VDD_DDR4: now also C222.1, C223.1, C224.1, C229.1, C230.1, C233.1, C236.1, C239.1, C241.1, C242.1, C250.1, R69.2, U13.A9 (VDDQ), U13.B9 (VDD), U13.C1 (VDDQ), U13.D1 (VDD), U13.D9 (VDDQ), U13.F2 (VDDQ), U13.F8 (VDDQ), U13.G1 (VDDQ), U13.G7 (VDD), U13.G9 (VDDQ), U13.J1 (VDD), U13.J2 (VDDQ), U13.J8 (VDDQ), U13.J9 (VDD), U13.L1 (VDD), U13.L9 (VDD), U13.R1 (VDD), U13.T9 (VDD)
- net at C248.1, R261.2: now also R267.2
