File: 13.kicad_sch (KiCad schematic)
At the start: 52 parts, among them J37 CON_SDCARD10_DM3BT-DSF-PEJS, U23 AM6442BSFGHAALV, U39 TPS22918DBVR, U44 MTFC16GAPALBH-IT, U49 TPD6E001RSER, U54 SN74LVC1G08DBVRE4, U86 SN74LVC1G11DCKR

Commit message: fix joint, offpage, and typo
DRC errors are cleared, some warnings remain.
Parts:
- removed *: MISTRAL_TITLEBLK_CSIZE, symbol 13-altium-import:root_0_MISTRAL_TITLEBLK_CSIZE
Connections:
- net DGND: now also C149.2, C428.2, C430.2, C437.2, C438.2, C443.2, J37.10, J37.11, J37.12 (CD2), J37.13, U44.A6 (VSS), U44.E7 (VSS), U44.G5 (VSS), U44.H10 (VSS), U44.J5 (VSS), U44.K8 (VSS), U44.N2 (VSSQ), U44.N5 (VSSQ), U44.P4 (VSSQ), U44.P6 (VSSQ)
- net GPIO_eMMC_RSTn: now also R196.1
- net MMC0_CLK: now also R456.2, R644.1
- net MMC0_DS: now also R444.2
- net MMC1_CLK: now also R645.1, R646.2
- net MMC1_CMD: now also R485.2
- net MMC1_D0: now also R479.2
- net MMC1_D1: now also R480.2
- net MMC1_D2: now also R483.2
- net MMC1_D3: now also R484.2
- net MMC1_SD_EN: now also R416.1
- net MMC1_SD_LS_EN: now also R426.2
- net SoC_MMC0_DAT0: now also R161.2
- net SoC_MMC0_DAT1: now also R163.2
- net SoC_MMC0_DAT2: now also R165.2
- net SoC_MMC0_DAT3: now also R159.2
- net SoC_MMC0_DAT4: now also R160.2
- net SoC_MMC0_DAT5: now also R162.2
- net SoC_MMC0_DAT6: now also R164.2
- net SoC_MMC0_DAT7: now also R166.2
- net VCC1V8: now also C170.1, C430.1, C443.1, R159.1, R160.1, R161.1, R162.1, R163.1, R164.1, R165.1, R166.1, R457.1, U44.C6 (VCCQ), U44.M4 (VCCQ), U44.N4 (VCCQ), U44.P3 (VCCQ)
- net VCC_3V3_SYS: now also C149.1, C150.1, C421.1, C437.1, C438.1, U39.1 (VIN), U44.F5 (VCC), U44.J10 (VCC), U44.K9 (VCC)
- net VDDIM: now also C427.1
- net VDDSHV_SD_IO: now also R479.1, R480.1, R483.1, R484.1, R485.1, TP39.1 (TP)
- net VDD_MMC1: now also FB9.1, U39.5 (QOD), U39.6 (VOUT)
- net VDD_MMC1_SD: now also C451.1
- net eMMC_RSTn: now also R193.2
