File: 14.kicad_sch (KiCad schematic)
At the start: 48 parts, among them Q18 BSS138LT1G, Q19 BSS138LT1G, U23 AM6442BSFGHAALV, U40 S28HS512TGABHM010, U85 SN74LVC1G08DBVRE4

Commit message: fix joint, offpage, and typo
DRC errors are cleared, some warnings remain.
Parts:
- removed *: MISTRAL_TITLEBLK_CSIZE, symbol 14-altium-import:root_0_MISTRAL_TITLEBLK_CSIZE
Connections:
- net DGND: now also C415.2, C418.2, C476.2, U40.B3 (VSS), U40.C1 (VSSQ)
- net GPIO_OSPI_RSTn: now also R429.1
- net OSPI_CLK: now also R167.1
- net OSPI_DQ0: now also R181.2
- net OSPI_DQ1: now also R176.2
- net OSPI_DQ2: now also R169.2
- net OSPI_DQ3: now also R172.2
- net OSPI_DQ4: now also R173.2
- net OSPI_DQ5: now also R180.2
- net OSPI_DQ6: now also R179.2
- net OSPI_DQ7: now also R178.2
- net OSPI_DQS: now also R154.1, R155.2
- net OSPI_DQS_SoC: now also R600.1
- net OSPI_RSTn: now also R414.1
- net TEST_LED1: now also R549.2
- net TEST_LED2: now also R554.2
- net VCC1V8: now also C415.1, C417.1, C418.1, C476.1, C477.1, R169.1, R172.1, R173.1, R176.1, R179.1, R180.1, R181.1, U40.D1 (VCCQ), U40.E4 (VCCQ)
