File: 15.kicad_sch (KiCad schematic)
At the start: 26 parts, among them U18 TMP100NA/3K, U29 TMP100NA/3K, U66 TCA9554APWR, U7 AT24CM01

Commit message: fix joint, offpage, and typo
DRC errors are cleared, some warnings remain.
Parts:
- removed *: MISTRAL_TITLEBLK_CSIZE, symbol 15-altium-import:root_0_MISTRAL_TITLEBLK_CSIZE
Connections:
- net DGND: now also R132.2, R17.1, R68.1, U66.2 (A1), U66.3 (A2)
- net EEPROM_A1: now also R26.2, R27.2
- net EEPROM_A2: now also R17.2, R18.2
- net TMP1_ADD0: now also R68.2, R72.2
- net TMP1_ADD1: now also R93.2, R98.2
- net TMP2_ADD0: now also R132.1, R133.2
- net TMP2_ADD1: now also R124.2, R125.2
- net VCC_3V3_SYS: now also C113.2, C209.1, C27.2, C53.2, R133.1, R18.1, R25.1, R72.1

Commit message: a lot, mpu power almost ready.
Parts:
- removed C209: 0.1uF, CAP0402_0-75, symbol 15-altium-import:root_1_CAP_Dup3
- removed R224, R226: 10K, RES0402_0-5, symbol 15-altium-import:root_2_RESISTOR_Dup6
- removed U66: TCA9554APWR, TSSOP16_25-59_205X180_1-2, symbol 15-altium-import:root_0_TCA9554APWR_TSSOP16
Connections:
- no-connect marks 8 -> 1
Other:
- note removed: "I2C ADDRESS: 0X38"
