File: 16.kicad_sch (KiCad schematic)
At the start: 69 parts, among them J14 CON_RJ45-14_LPJG16314A4NL, Q12 BSS138LT1G, Q13 BSS138LT1G, Q3 BSS138LT1G, U15 DP83867IRRGZ, U69 SN74LVC1G08DBVRE4, U75 TS3DDR3812RUAR

Commit message: fix joint, offpage, and typo
DRC errors are cleared, some warnings remain.
Parts:
- removed *: MISTRAL_TITLEBLK_CSIZE, symbol 16-altium-import:root_0_MISTRAL_TITLEBLK_CSIZE
Connections:
- net CPSW_EARTH: now also C287.1, J14.16 (SH2), R299.1
- net CPSW_ETH1_GPIO_0: now also R251.1, R41.2
- net CPSW_ETH1_GPIO_1: now also R35.2, R36.1
- net CPSW_ETH1_LED2: now also R234.1
- net CPSW_ETH1_LED3: now also R37.1
- net CPSW_ETH1_LED_1000: now also R31.1, R32.2
- net CPSW_ETH1_LED_ACT: now also R33.2, R34.1
- net CPSW_FET_SEL: now also U75.10 (SEL2)
- net CPSW_RGMII1_RD0: now also R54.1, R56.2
- net CPSW_RGMII1_RD2: now also R51.2, R52.1
- net CPSW_RGMII1_RESETn: now also R240.1
- net CPSW_RGMII1_RX_CTL: now also R249.1, R39.1
- net DGND: now also C237.2, C238.2, C249.2, C253.2, C258.2, C259.2, C260.2, C261.2, C266.2, C274.2, C281.2, C284.2, C35.2, C36.2, C39.2, C41.2, C43.2, C44.2, C51.2, C52.2, R241.2, R249.2, R251.2, R299.2, R31.2, R34.2, R52.2, R54.2
- net GPIO_CPSW1_RST: now also R242.1
- net VCC_3V3_SYS: now also C220.1, C237.1, C260.1, C266.1, C276.1, C281.1, C284.1, C35.1, C44.1, C52.1, R32.1, R33.1, R35.1, R39.2, R41.1, R51.1, R79.2, R81.1, U15.19 (VDDIO), U15.30 (VDDIO), U75.1 (VCC), U75.17 (VCC)
- net VDD_1V0: now also C238.1, C253.1, C259.1, C263.1, C274.1, C36.1, C39.1, C41.1, U15.24 (VDD1P0), U15.31 (VDD1P0), U15.6 (VDD1P0)
- net VDD_2V5: now also C249.1, C258.1, C261.1, C43.1, U15.3 (VDDA2P5)
- net at U15.13 (VDDA1P8): now also TP11.1 (TP), U15.48 (VDDA1P8)
- net PRG0_PRU1_GPO7/CPSW_RGMII1_RD0 renamed PRG0_PRU1_GPO7/CPSW_RGMII1_RD0
- no-connect marks 25 -> 23

Commit message: a lot, mpu power almost ready.
Parts:
- removed C260, C276, C284: 0.1uF, CAP0402_0-75, symbol 16-altium-import:root_0_CAP_Dup3
- removed R278, R292: 10K, RES0402_0-5, symbol 16-altium-import:root_0_RESISTOR_Dup6
- removed U75: TS3DDR3812RUAR, TQFN42_19-68_140X360_0-8, symbol 16-altium-import:root_0_TS3DDR3812RUAR_WQFN42
Connections:
- no-connect marks 23 -> 5
