File: 20.kicad_sch (KiCad schematic)
At the start: 74 parts, among them J30 HDR_2X1, SW2 218-8LPSTR, SW3 218-8LPSTR, U79 SN74AVC8T245RHL, U81 SN74AVC8T245RHL, U90 SN74LVC1G08DBVRE4, U96 TCA6424ARGJR

Commit message: fix joint, offpage, and typo
DRC errors are cleared, some warnings remain.
Parts:
- removed *: MISTRAL_TITLEBLK_CSIZE, symbol 20-altium-import:root_0_MISTRAL_TITLEBLK_CSIZE
Connections:
- net PORZ_OUT is gone; now on net PORz_OUT: R434.2
- net BOOTMODEON: now also R453.1
- net DGND: now also R473.2, R488.2, R489.2, R497.2, R498.2, R502.2, R503.2, R509.2, R510.2, R513.2, R514.2, R518.2, R519.2, R529.2, U79.11 (GND1), U79.12 (GND2), U79.13 (GND3), U81.11 (GND1), U81.12 (GND2), U81.13 (GND3), U96.25 (GND), U96.33 (EP)
- net DIR: now also R355.1, R356.2
- net SYS_BOOTMODE0: now also R529.1, SW2.1
- net SYS_BOOTMODE1: now also R519.1, SW2.2
- net SYS_BOOTMODE10: now also R497.1, SW3.3
- net SYS_BOOTMODE11: now also R502.1, SW3.4
- net SYS_BOOTMODE12: now also R509.1, SW3.5
- net SYS_BOOTMODE13: now also R513.1, SW3.6
- net SYS_BOOTMODE14: now also R518.1, SW3.7
- net SYS_BOOTMODE15: now also R528.1, SW3.8
- net SYS_BOOTMODE2: now also R514.1, SW2.3
- net SYS_BOOTMODE3: now also R510.1, SW2.4
- net SYS_BOOTMODE4: now also R503.1, SW2.5
- net SYS_BOOTMODE5: now also R498.1, SW2.6
- net SYS_BOOTMODE6: now also R489.1, SW2.7
- net SYS_BOOTMODE7: now also R474.1, SW2.8
- net SYS_BOOTMODE8: now also R473.1, SW3.1
- net SYS_BOOTMODE9: now also R488.1, SW3.2
- net TEST_GPIO3: now also R439.2
- net VCC3V3_TA: now also C190.2, C388.1, C405.1, C434.1, U96.27 (VCCP), U96.31 (VCC)
- net VCC_3V3_SYS: now also R475.2, R487.2, R490.2, R496.2, R499.2, R501.2, R504.2, R508.2, R511.2, R512.2, R515.2, R517.2, R520.2, R527.2, U79.23 (VCCB1), U81.23 (VCCB1)

Commit message: a lot, mpu power almost ready.
Parts:
- removed C190: 0.01uF, CAP0402N, symbol 20-altium-import:root_3_CAP_Dup2
- removed C384, C388, C404, C405: 0.1uF, CAP0402_0-75, symbol 20-altium-import:root_0_CAP_Dup3
- removed C434: 0.1uF, CAP0402_0-75, symbol 20-altium-import:root_1_CAP_Dup3
- removed J30: HDR_2X1, HDR_2X1_100_S_T_10-8, symbol 20-altium-import:root_0_HEADER_2X1_Dup1
- removed R355, R356, R532, R533: 10K, RES0402_0-5, symbol 20-altium-import:root_2_RESISTOR_Dup6
- removed R434, R435, R454: 0E, RES0402_0-5, symbol 20-altium-import:root_3_RESISTOR_Dup5
- removed R439, R453: 10K, RES0402_0-5, symbol 20-altium-import:root_0_RESISTOR_Dup6
- removed R555: 1K_1%, RES0402_0-5, symbol 20-altium-import:root_2_RESISTOR_Dup5
- removed TP42, TP43: TP20_SMD, TP20_SMD, symbol 20-altium-import:root_0_TESTPOINT
- removed U79, U81: SN74AVC8T245RHL, QFN24_19-68_220X140_1, symbol 20-altium-import:root_0_SN74AVC8T245RHL_QFN24
- removed U90: SN74LVC1G08DBVRE4, SOT23-5, symbol 20-altium-import:root_0_SN74LVC1G08DBVRE4_SOT23-5
- removed U96: TCA6424ARGJR, QFN32_19-68_200X200, symbol 20-altium-import:root_0_TCA6424ARGJR_QFN32
Connections:
- net SYS_BOOTMODE0: now also R325.2
- net SYS_BOOTMODE1: now also R326.2
- net SYS_BOOTMODE10: now also R374.2
- net SYS_BOOTMODE11: now also R375.2
- net SYS_BOOTMODE12: now also R376.2
- net SYS_BOOTMODE13: now also R377.2
- net SYS_BOOTMODE14: now also R378.2
- net SYS_BOOTMODE15: now also R379.2
- net SYS_BOOTMODE2: now also R327.2
- net SYS_BOOTMODE3: now also R328.2
- net SYS_BOOTMODE4: now also R329.2
- net SYS_BOOTMODE5: now also R330.2
- net SYS_BOOTMODE6: now also R331.2
- net SYS_BOOTMODE7: now also R332.2
- net SYS_BOOTMODE8: now also R372.2
- net SYS_BOOTMODE9: now also R373.2
- no-connect marks 8 -> 0
Other:
- note removed: "I2C ADDRESS: 0x22"
