File: 21.kicad_sch (KiCad schematic)
At the start: 61 parts, among them J11 HDR_2X1, J13 HDR_2X1, J19 HDR_2X1, J20 HDR_2X1, J22 HDR_2X1, J4 HDR_1X5, J8 HDR_2X1, U1 INA226AIDGSR, U11 INA226AIDGSR, U14 INA226AIDGSR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

Commit message: fix joint, offpage, and typo
DRC errors are cleared, some warnings remain.
Parts:
- removed *: MISTRAL_TITLEBLK_CSIZE, symbol 21-altium-import:root_0_MISTRAL_TITLEBLK_CSIZE
Connections:
- net DGND: now also U14.1 (A1), U16.2 (A0), U6.1 (A1)
- net INA_ALERT: now also R47.1
- net SOC_DVDD1V8: now also J13.2
- net SoC_DVDD3V3: now also J19.2
- net SoC_I2C1_SCL: now also U11.2 (A0), U16.1 (A1), U28.1 (A1)
- net SoC_I2C1_SDA: now also U1.2 (A0), U11.1 (A1), U28.2 (A0)
- net VCC1V2_DDR: now also C21.2, J8.1
- net VCC1V8: now also J13.1
- net VCC_3V3_SYS: now also C10.1, C109.1, C17.1, C32.1, C45.1, C50.1, C55.2, J19.1, R265.1
- net VCC_CORE: now also C72.2, J20.1
- net VDDA1V8: now also C117.2, J22.1
- net VDDAR_CORE: now also J11.2
- net VDDA_1V8: now also J22.2
- net VDD_0V85: now also C31.2, J11.1
- net VDD_CORE: now also J20.2
- net VDD_DDR4: now also J8.2
- net at R229.1, U11.9 (VIN-): now also C214.2, U11.8 (VBUS)
- net at C203.1: now also R10.1, U1.10 (VIN+)
- net at C203.2: now also R11.1, U1.8 (VBUS), U1.9 (VIN-)
- net at R350.1, U28.9 (VIN-): now also C393.2, U28.8 (VBUS)
- net at C393.1: now also R352.1, U28.10 (VIN+)
- net at R216.1, U6.9 (VIN-): now also C204.2, U6.8 (VBUS)
- net at R215.1, U6.10 (VIN+): now also C204.1
- net at R73.1, U14.9 (VIN-): now also C47.2, U14.8 (VBUS)
- net at C214.1: now also R228.1, U11.10 (VIN+)
- net at R280.1, U16.10 (VIN+): now also C269.1
- net at R281.1, U16.9 (VIN-): now also C269.2, U16.8 (VBUS)
- net at R74.1, U14.10 (VIN+): now also C47.1

Commit message: a lot, mpu power almost ready.
Parts:
- removed C10, C109, C17, C203, C204, C214, C269, C32, C393, C45, C47, C50: 0.1uF, CAP0402_0-75, symbol 21-altium-import:root_0_CAP_Dup3
- removed C117, C21, C221, C31, C55, C72: 0.1uF, CAP0402_0-75, symbol 21-altium-import:root_1_CAP_Dup3
- removed J11, J13, J19, J20, J22, J8: HDR_2X1, HDR_2X1_100_S_T_10-8, symbol 21-altium-import:root_0_HEADER_2X1_Dup1
- removed J4: HDR_1X5, HDR_5X1_100_S_T_11-2, symbol 21-altium-import:root_0_mirrored_HEADER_5X1
- removed R1, R12, R122, R13, R244, R28, R43, R48: 0E, RES0402_0-5, symbol 21-altium-import:root_1_RESISTOR_Dup5
- removed R10, R11, R215, R216, R228, R229, R280, R281, R350, R352, R73, R74: 10E_1%, RES0402_0-5, symbol 21-altium-import:root_3_RESISTOR_Dup6
- removed R22: 0.01E_0.5%, RES1206-4TERM_0-75, symbol 21-altium-import:root_3_mirrored_RESISTOR-4TERM
- removed R227, R295: 0.01E_0.5%, RES1206-4TERM_0-75, symbol 21-altium-import:root_1_RESISTOR-4TERM
- removed R233, R351: 0.01E_0.5%, RES1206-4TERM_0-75, symbol 21-altium-import:root_3_RESISTOR-4TERM
- removed R47: 10K_1%, RES0402N, symbol 21-altium-import:root_2_mirrored_RESISTOR_Dup3
- removed R92: 0.002E_1%, RES2512-4TERM_0-75, symbol 21-altium-import:root_1_mirrored_RESISTOR-4TERM
- removed U1, U11, U14, U16, U28, U6: INA226AIDGSR, MSOP10_19-68_120X120_1-1, symbol 21-altium-import:root_0_INA226AIDGS_MSOP10
Connections:
- no-connect marks 2 -> 0
Other:
- note removed: "I2C ADDRESS: 0x40"
- note removed: "I2C ADDRESS: 0x41"
- note removed: "I2C ADDRESS: 0x46"
- note removed: "I2C ADDRESS: 0x4B"
- note removed: "I2C ADDRESS: 0x4C"
- note removed: "I2C ADDRESS: 0x4E"
