File: 23.kicad_sch (KiCad schematic)
At the start: 42 parts, among them J39 HDR_2X1, J40 HDR_2X1, U23 AM6442BSFGHAALV, U37 SN74AVC4T245RGYR, U45 TXS0102DCUR, U46 SN74AVC2T244DQMR, U47 SN74LVC1G04DCKR, U55 TXS0102DCUR, U56 SN74AVC2T244DQMR, U98 SN74AVC4T245RGYR

Commit message: fix joint, offpage, and typo
DRC errors are cleared, some warnings remain.
Parts:
- removed *: MISTRAL_TITLEBLK_CSIZE, symbol 23-altium-import:root_0_MISTRAL_TITLEBLK_CSIZE
Connections:
- net DGND: now also C145.1, C157.1, C162.1, R183.2, U37.8 (GND1), U37.9 (GND2), U98.8 (GND1), U98.9 (GND2)
- net JTAG_DIR: now also U37.3 (2DIR)
- net SEL_XDS: now also U98.14 (~{2OE})
- net SEL_XDS110_INV: now also U37.14 (~{2OE})
- net SoC_EMU0: now also J39.1, R634.2
- net SoC_EMU1: now also J40.1, R635.2
- net VCC_3V3_SYS: now also C145.2, C157.2, C162.2, C165.2, U37.1 (VCCA), U45.3 (VCCA), U46.1 (VCCA)
- net XDS110_DIR: now also U98.3 (2DIR)

Commit message: a lot, mpu power almost ready.
Parts:
- removed C145, C146, C155, C156, C157, C162, C165, C171, C178, C188, C189, C461, C464: 0.1uF, CAP0402_0-75, symbol 23-altium-import:root_2_CAP_Dup3
- removed J39, J40: HDR_2X1, HDR_2X1_100_S_T_10-8, symbol 23-altium-import:root_0_HEADER_2X1_Dup1
- removed R147, R506: 22E_1%, RES0402_0-5, symbol 23-altium-import:root_1_mirrored_RESISTOR_Dup5
- removed R148, R184, R507, R643: 10K, RES0402_0-5, symbol 23-altium-import:root_2_RESISTOR_Dup6
- removed R183, R634, R635, R640, R641, R642: 10K, RES0402_0-5, symbol 23-altium-import:root_0_RESISTOR_Dup6
- removed R455, R458: 4.7K, RES0402_0-5, symbol 23-altium-import:root_0_RESISTOR_Dup4
- removed R630, R631: 1K_1%, RES0402_0-5, symbol 23-altium-import:root_2_RESISTOR_Dup5
- removed U37, U98: SN74AVC4T245RGYR, QFN16_19-68_160X140, symbol 23-altium-import:root_0_SN74AVC4T245RGYR_QFN16
- removed U45, U55: TXS0102DCUR, VSSOP8_19-68_85X95_0-9, symbol 23-altium-import:root_0_TXS0102DCUR_VSSOP8
- removed U46, U56: SN74AVC2T244DQMR, X2SON8_15-74_70X50, symbol 23-altium-import:root_0_SN74AVC2T244DQMR_X2SON8
- removed U47: SN74LVC1G04DCKR, SC70-5, symbol 23-altium-import:root_0_SN74LVC1G04DCKR_SC70-5
- added C144, C529: 100n,±10%,16V, Abacus:C_0402_1005Metric_for_0.25mm_grid, symbol JLC_C0402:100n,±10%,16V
- added J25: HDR_2X10, HDR_2X10_FTR-110-51-D-06_S_S_8-7, symbol 24-altium-import:root_0_HEADER_10X2_FTR-06
- added R150, R411, R460, R461: 4.7k,1%, Abacus:R_0402_1005Metric_for_0.25mm_grid, symbol JLC_R0402:4.7k,1%
- added R177: 0R,1%, Abacus:R_0402_1005Metric_for_0.25mm_grid, symbol JLC_R0402:0R,1%
- added R409, R410: 22R,1%, Abacus:R_0402_1005Metric_for_0.25mm_grid, symbol JLC_R0402:22R,1%
- added R685: 100R,1%, Abacus:R_0402_1005Metric_for_0.25mm_grid, symbol JLC_R0402:100R,1%
Connections:
- net SoC_EMU0 is gone; now on net JTAG_EMU0: U23.D10 (EMU0)
- net SoC_EMU1 is gone; now on net JTAG_EMU1: U23.E10 (EMU1)
- net SoC_TCK is gone; now on net JTAG_TCK: U23.B11 (TCK)
- net SoC_TDI is gone; now on net JTAG_TDI: U23.C11 (TDI)
- net SoC_TDO is gone; now on net JTAG_TDO: R323.1
- net SoC_TMS is gone; now on net JTAG_TMS: U23.C12 (TMS)
- net SoC_TRST# is gone; now on net JTAG_TRST#: R322.1, U23.D11 (TRSTN)
- net DGND: now also C144.2, C529.2, J25.10, J25.12, J25.16, J25.20, R177.2, R411.2
- net JTAG_EMU0: now also J25.13, R460.2
- net JTAG_EMU1: now also J25.14, R461.2
- net JTAG_TCK: now also R409.2, R410.2
- net JTAG_TDI: now also J25.3
- net JTAG_TDO: now also J25.7
- net JTAG_TMS: now also J25.1
- net JTAG_TRST#: now also C529.1, R411.1, R685.2
- net VCC_3V3_SYS: now also C144.1, J25.5, R150.1, R460.1, R461.1
- new net: J25.11, R409.1
- new net: J25.2, R685.1
- new net: J25.9, R410.1
- new net JTAG_EMU_RSTn: J25.15, R150.2
- new net JTAG_TDIS: J25.4, R177.1
- no-connect marks 1 -> 4
Other:
- note added: "JTAG 20 PIN cTI CONNECTOR"
- note added: "https://software-dl.ti.com/ccs/esd/documents/xdsdebugprobes/emu_xds_target_connection_guide.html"
- note removed: "BUFFER 20 PIN JTAG"
- note removed: "BUFFER XDS110"
- note removed: "JTAG BUFFER"
- note removed: "Off Page Connections"
- moved on the sheet: R322, R323, U23B
