File: 24.kicad_sch (KiCad schematic)
At the start: 49 parts, among them J25 HDR_2X10, J29 HDR_1X3, J33 CON_PMC_2X30_F, U48 TXS0102DCUR, U52 SN74LVC1G32DBVR, U53 SN74LVC1G32DBVR, U60 SN74CB3Q3257PWR, U93 SN74LVC1G32DBVR, U94 SN74LVC1G32DBVR

Commit message: fix joint, offpage, and typo
DRC errors are cleared, some warnings remain.
Parts:
- removed *: MISTRAL_TITLEBLK_CSIZE, symbol 24-altium-import:root_0_MISTRAL_TITLEBLK_CSIZE
Connections:
- net DGND: now also C163.1, C164.1, J25.12, J25.16, J25.20, J33.61, J33.62, J33.63, U60.12 (4A), U60.9 (3A)
- net JTAG_MIPI_RTCK: now also R639.1
- net JTAG_MIPI_TCK: now also R187.1
- net JTAG_cTI_RTCK: now also R636.1, R637.1
- net JTAG_cTI_TCK: now also R188.1
- net VCC_3V3_MIPI: now also R460.1
- net VCC_3V3_SYS: now also C144.2, C182.2, C183.2, C194.2, C411.2, C456.2, C457.2

Commit message: a lot, mpu power almost ready.
Parts:
- removed C144, C194, C529: 0.1uF, CAP0402_0-75, symbol 24-altium-import:root_2_CAP_Dup3
- removed C168, C169: 8.2pF, CAP0402_0-75, symbol 24-altium-import:root_0_CAP_Dup3
- removed C182, C183, C456, C457: 0.01uF, CAP0402N, symbol 24-altium-import:root_1_CAP_Dup2
- removed J25: HDR_2X10, HDR_2X10_FTR-110-51-D-06_S_S_8-7, symbol 24-altium-import:root_0_HEADER_10X2_FTR-06
- removed J29: HDR_1X3, HDR_3X1_100_S_T, symbol 24-altium-import:root_0_HEADER_3X1
- removed J33: CON_PMC_2X30_F, CON_PMC2X30_QSH-030-01-D-A_S_S_S_3-3, symbol 24-altium-import:root_0_CON_PMC_30X2_F
- removed R150: 4.7K, RES0402_0-5, symbol 24-altium-import:root_0_RESISTOR_Dup4
- removed R177: 0E, RES0402_0-5, symbol 24-altium-import:root_2_RESISTOR_Dup5
- removed R187, R188, R637, R639: 10K, RES0402_0-5, symbol 24-altium-import:root_2_RESISTOR_Dup6
- removed R189, R190, R636, R638: 100E, RES0402_0-5, symbol 24-altium-import:root_0_RESISTOR_Dup6
- removed R194, R195, R491, R492: 33E_1%, RES0402_0-5, symbol 24-altium-import:root_1_RESISTOR_Dup6
- removed R685: 100E, RES0402N, symbol 24-altium-import:root_1_RESISTOR_Dup2
- removed U52, U53, U93, U94: SN74LVC1G32DBVR, SOT23-5_1-5, symbol 24-altium-import:root_0_mirrored_SN74LVC1G32DBVR_SOT23-5
- removed U60: SN74CB3Q3257PWR, TSSOP16_25-59_205X180, symbol 24-altium-import:root_0_SN74CB3Q3257PWR_TSSOP16
Connections:
- no-connect marks 28 -> 4
Other:
- note removed: "From SoC GPMC"
- note removed: "JTAG 20 PIN cTI CONNECTOR"
- note removed: "JTAG CLOCK BUFFER"
- note removed: "MIPI 60 PIN CONNECTOR"
