File: 27.kicad_sch (KiCad schematic)
At the start: 27 parts, among them J15 HDR_2X1, J16 HDR_2X1, J17 HDR_2X1, J18 HDR_2X1, J2 CON_XMC_5X30_F, U2 TPS22919DCKR, U23 AM6442BSFGHAALV, U63 TPS22919DCKR, U64 TPS22919DCKR

Commit message: fix joint, offpage, and typo
DRC errors are cleared, some warnings remain.
Parts:
- removed *: MISTRAL_TITLEBLK_CSIZE, symbol 27-altium-import:root_0_MISTRAL_TITLEBLK_CSIZE
Connections:
- net DGND: now also C12.2, C14.2, C206.2, J2.A10, J2.A16, J2.A18, J2.A24, J2.A25, J2.B10, J2.B16, J2.B19, J2.B23, J2.B25, J2.B26, J2.B27, J2.B30, J2.B5, J2.B6, J2.C10, J2.C13, J2.C17, J2.C18, J2.C20, J2.C25, J2.C7, J2.D10, J2.D13, J2.D16, J2.D20, J2.D25, J2.D30, J2.D7, J2.E10, J2.E16, J2.E20, J2.E22, J2.E25, J2.E28, J2.E29, J2.E6, J2.E7
- net VCC1V8: now also U63.1 (IN), U63.3 (ON)
- net VCC1V8_HSE: now also C206.1, J2.C2, U63.5 (QOD), U63.6 (OUT)
- net VCC3V3_IO_HSE: now also C14.1, J2.A28, J2.A29, U64.5 (QOD), U64.6 (OUT)
- net VCC_3V3_SYS: now also U64.1 (IN), U64.3 (ON)
- net VCC_5V0: now also U2.1 (IN), U2.3 (ON)
- net VCC_5V0_HSE: now also C12.1, J2.A1, J2.A2, U2.5 (QOD), U2.6 (OUT)

Commit message: a lot, mpu power almost ready.
Parts:
- removed C11, C15, C16, C18, C212, C216: 1uF, CAP0402_0-75, symbol 27-altium-import:root_0_CAP_Dup3
- removed C12, C13, C14, C19, C205, C206: 0.1uF, CAP0402_0-75, symbol 27-altium-import:root_0_CAP_Dup3
- removed J15, J16, J17, J18: HDR_2X1, HDR_2X1_100_S_T, symbol 27-altium-import:root_0_HEADER_2X1
- removed J2: CON_XMC_5X30_F, CON_XMC5X30_SEAF-30-06-05-2-A_S_S_S_6-4, symbol 27-altium-import:root_0_CON_XMC30X5_F_SEAF
- removed U2, U63, U64: TPS22919DCKR, SC70-6_1-1, symbol 27-altium-import:root_0_TPS22919_SC70-6
Connections:
- net PRG0_MDIO0_MDC: no longer names the net of U23.P3 (PRG0_MDIO0_MDC)
- net PRG0_PRU0GPO0: no longer names the net of U23.Y1 (PRG0_PRU0_GPO0)
- net PRG0_PRU0GPO1: no longer names the net of U23.R4 (PRG0_PRU0_GPO1)
- net PRG0_PRU0GPO11: no longer names the net of U23.Y3 (PRG0_PRU0_GPO11)
- net PRG0_PRU0GPO12: no longer names the net of U23.AA3 (PRG0_PRU0_GPO12)
- net PRG0_PRU0GPO13: no longer names the net of U23.R6 (PRG0_PRU0_GPO13)
- net PRG0_PRU0GPO14: no longer names the net of U23.V4 (PRG0_PRU0_GPO14)
- net PRG0_PRU0GPO15: no longer names the net of U23.T5 (PRG0_PRU0_GPO15)
- net PRG0_PRU0GPO16: no longer names the net of U23.U4 (PRG0_PRU0_GPO16)
- net PRG0_PRU0GPO17: no longer names the net of U23.U1 (PRG0_PRU0_GPO17)
- net PRG0_PRU0GPO18: no longer names the net of U23.V1 (PRG0_PRU0_GPO18)
- net PRG0_PRU0GPO19: no longer names the net of U23.W1 (PRG0_PRU0_GPO19)
- net PRG0_PRU0GPO2: no longer names the net of U23.U2 (PRG0_PRU0_GPO2)
- net PRG0_PRU0GPO3: no longer names the net of U23.V2 (PRG0_PRU0_GPO3)
- net PRG0_PRU0GPO4: no longer names the net of U23.AA2 (PRG0_PRU0_GPO4)
- net PRG0_PRU0GPO5: no longer names the net of U23.R3 (PRG0_PRU0_GPO5)
- net PRG0_PRU0GPO6: no longer names the net of U23.T3 (PRG0_PRU0_GPO6)
- net PRG0_PRU0GPO7: no longer names the net of U23.T1 (PRG0_PRU0_GPO7)
- net PRG0_PRU0GPO8: no longer names the net of U23.T2 (PRG0_PRU0_GPO8)
- net PRG0_PRU0_GPO10/CPSW_RGMII1_RXC renamed CPSW_RGMII1_RXC
- net PRG0_PRU0_GPO9/CPSW_RGMII1_RX_CTL renamed CPSW_RGMII1_RX_CTL
- net PRG0_PRU1GPO0: no longer names the net of U23.Y2 (PRG0_PRU1_GPO0)
- net PRG0_PRU1GPO1: no longer names the net of U23.W2 (PRG0_PRU1_GPO1)
- net PRG0_PRU1GPO11: no longer names the net of U23.W4 (PRG0_PRU1_GPO11)
- net PRG0_PRU1GPO12: no longer names the net of U23.Y4 (PRG0_PRU1_GPO12)
- net PRG0_PRU1GPO13: no longer names the net of U23.T6 (PRG0_PRU1_GPO13)
- net PRG0_PRU1GPO14: no longer names the net of U23.U6 (PRG0_PRU1_GPO14)
- net PRG0_PRU1GPO15: no longer names the net of U23.U5 (PRG0_PRU1_GPO15)
- net PRG0_PRU1GPO16: no longer names the net of U23.AA4 (PRG0_PRU1_GPO16)
- net PRG0_PRU1GPO2: no longer names the net of U23.V3 (PRG0_PRU1_GPO2)
- net PRG0_PRU1GPO3: no longer names the net of U23.T4 (PRG0_PRU1_GPO3)
- net PRG0_PRU1GPO4: no longer names the net of U23.W3 (PRG0_PRU1_GPO4)
- net PRG0_PRU1GPO5: no longer names the net of U23.P4 (PRG0_PRU1_GPO5)
- net PRG0_PRU1GPO6: no longer names the net of U23.R5 (PRG0_PRU1_GPO6)
- net PRG0_PRU1GPO8: no longer names the net of U23.R1 (PRG0_PRU1_GPO8)
- net PRG0_PRU1_GPO10/CPSW_RGMII1_RD2 renamed CPSW_RGMII1_RD2
- net PRG0_PRU1_GPO17/CPSW_RGMII1_RD3 renamed CPSW_RGMII1_RD3
- net PRG0_PRU1_GPO7/CPSW_RGMII1_RD0 renamed CPSW_RGMII1_RD0
- net PRG0_PRU1_GPO9/CPSW_RGMII1_RD1 renamed CPSW_RGMII1_RD1
- net PRG1_ETH2_LED_1000/RX_ER: no longer names the net of U23.AA13 (PRG1_PRU1_GPO5)
- net PRG1_ETH2_LED_LINK: no longer names the net of U23.U12 (PRG1_PRU1_GPO8)
- net PRG1_ETH3_LED_1000/RX_ER: no longer names the net of U23.V13 (PRG1_PRU0_GPO5)
- net PRG1_ETH3_LED_LINK: no longer names the net of U23.W13 (PRG1_PRU0_GPO8)
- net PRG1_IEP0_EDC_LATCH_IN0: no longer names the net of U23.V7 (PRG1_PRU0_GPO18)
- net PRG1_IEP0_EDC_LATCH_IN1: no longer names the net of U23.U13 (PRG1_PRU0_GPO7)
- net PRG1_IEP0_EDC_SYNC_OUT0: no longer names the net of U23.W7 (PRG1_PRU0_GPO19)
- net PRG1_IEP0_EDC_SYNC_OUT2: no longer names the net of U23.U7 (PRG1_PRU0_GPO17)
- net PRG1_PRU1GPO18: no longer names the net of U23.Y13 (PRG1_PRU1_GPO18)
- net PRG1_PRU1GPO19: no longer names the net of U23.V12 (PRG1_PRU1_GPO19)
- net PRG1_RGMII1_RD0: no longer names the net of U23.Y7 (PRG1_PRU0_GPO0)
- net PRG1_RGMII1_RD1: no longer names the net of U23.U8 (PRG1_PRU0_GPO1)
- net PRG1_RGMII1_RD2: no longer names the net of U23.W8 (PRG1_PRU0_GPO2)
- net PRG1_RGMII1_RD3: no longer names the net of U23.V8 (PRG1_PRU0_GPO3)
- net PRG1_RGMII1_RXC: no longer names the net of U23.AA7 (PRG1_PRU0_GPO6)
- net PRG1_RGMII1_RX_CTL: no longer names the net of U23.Y8 (PRG1_PRU0_GPO4)
- net PRG1_RGMII1_TD0: no longer names the net of U23.AA8 (PRG1_PRU0_GPO11)
- net PRG1_RGMII1_TD1: no longer names the net of U23.U9 (PRG1_PRU0_GPO12)
- net PRG1_RGMII1_TD2: no longer names the net of U23.W9 (PRG1_PRU0_GPO13)
- net PRG1_RGMII1_TD3: no longer names the net of U23.AA9 (PRG1_PRU0_GPO14)
- net PRG1_RGMII1_TXC: no longer names the net of U23.V9 (PRG1_PRU0_GPO16)
- net PRG1_RGMII1_TX_CTL: no longer names the net of U23.Y9 (PRG1_PRU0_GPO15)
- net PRG1_RGMII2_RD0: no longer names the net of U23.W11 (PRG1_PRU1_GPO0)
- net PRG1_RGMII2_RD1: no longer names the net of U23.V11 (PRG1_PRU1_GPO1)
- net PRG1_RGMII2_RD2: no longer names the net of U23.AA12 (PRG1_PRU1_GPO2)
- net PRG1_RGMII2_RD3: no longer names the net of U23.Y12 (PRG1_PRU1_GPO3)
- net PRG1_RGMII2_RXC: no longer names the net of U23.U11 (PRG1_PRU1_GPO6)
- net PRG1_RGMII2_RX_CTL: no longer names the net of U23.W12 (PRG1_PRU1_GPO4)
- net PRG1_RGMII2_TD0: no longer names the net of U23.AA10 (PRG1_PRU1_GPO11)
- net PRG1_RGMII2_TD1: no longer names the net of U23.V10 (PRG1_PRU1_GPO12)
- net PRG1_RGMII2_TD2: no longer names the net of U23.U10 (PRG1_PRU1_GPO13)
- net PRG1_RGMII2_TD3: no longer names the net of U23.AA11 (PRG1_PRU1_GPO14)
- net PRG1_RGMII2_TXC: no longer names the net of U23.Y10 (PRG1_PRU1_GPO16)
- net PRG1_RGMII2_TX_CTL: no longer names the net of U23.Y11 (PRG1_PRU1_GPO15)
- no-connect marks 7 -> 67
Other:
- note removed: "HSE CONNECTOR LOAD SWITCHES"
- note removed: "LOAD SWITCH RATING 1.8V, 1.5A"
- note removed: "LOAD SWITCH RATING 3.3V, 1.5A"
- note removed: "LOAD SWITCH RATING 5V, 1.5A"
- note removed: "SYNC TP"
