File: 28.kicad_sch (KiCad schematic)
At the start: 18 parts, among them J7 HDR_2X5, U23 AM6442BSFGHAALV, U8 TS3A27518ERTWR

Commit message: fix joint, offpage, and typo
DRC errors are cleared, some warnings remain.
Parts:
- removed *: MISTRAL_TITLEBLK_CSIZE, symbol 28-altium-import:root_0_MISTRAL_TITLEBLK_CSIZE
Connections:
- net BOOTMODE0: now also RA2.1
- net BOOTMODE1: now also RA2.2
- net BOOTMODE10: now also RA4.3
- net BOOTMODE11: now also RA4.4
- net BOOTMODE12: now also RA4.5
- net BOOTMODE13: now also RA4.6
- net BOOTMODE14: now also RA4.7
- net BOOTMODE15: now also RA4.8
- net BOOTMODE2: now also RA2.3
- net BOOTMODE3: now also RA2.4
- net BOOTMODE4: now also RA2.5
- net BOOTMODE5: now also RA2.6
- net BOOTMODE6: now also RA2.7
- net BOOTMODE7: now also RA2.8
- net BOOTMODE8: now also RA4.1
- net BOOTMODE9: now also RA4.2
- net DGND: now also U8.2 (GND), U8.25 (PAD)
- net FSI_FET_SEL: now also U8.21 (IN1)
- net GPMC0_ADVn_ALE: now also RA6.2
- net GPMC0_BE0n_CLE: now also RA6.5
- net GPMC0_BE1n: now also RA6.6
- net GPMC0_CLK: now also RA6.1
- net GPMC0_CSn0: now also R391.1
- net GPMC0_OEn_REn: now also RA6.3
- net GPMC0_WAIT0: now also RA6.7
- net GPMC0_WAIT1: now also RA6.8
- net GPMC0_WEn: now also RA6.4
- net GPMC0_WPn: now also R392.1
- net VCC_3V3_SYS: now also C26.1, C29.1

Commit message: a lot, mpu power almost ready.
Parts:
- removed C26, C29: 0.1uF, CAP0402_0-75, symbol 28-altium-import:root_0_CAP_Dup3
- removed J7: HDR_2X5, HDR_5X2_100_S_T_8-6, symbol 28-altium-import:root_0_HEADER_5X2
- removed R21, R218: 10K, RES0402_0-5, symbol 28-altium-import:root_0_mirrored_RESISTOR_Dup6
- removed R390, R391, R392, R393: 0E, RES0402_0-5, symbol 28-altium-import:root_1_RESISTOR_Dup5
- removed RA1, RA2, RA3, RA4, RA5, RA6: 0E, RESA_EXB2HV_0602-8_0-6, symbol 28-altium-import:root_1_mirrored_RESARR_ISO8_0402
- removed U8: TS3A27518ERTWR, QFN24_19-68_160X160_0-8, symbol 28-altium-import:root_0_TS3A27518ERTWR_QFN24
Connections:
- net GPMC0_ADVn_ALE: no longer names the net of U23.P16 (GPMC0_ADVN_ALE)
- net GPMC0_BE0n_CLE: no longer names the net of U23.P17 (GPMC0_BE0N_CLE)
- net GPMC0_BE1n: no longer names the net of U23.T19 (GPMC0_BE1N)
- net GPMC0_CLK: no longer names the net of U23.R17 (GPMC0_CLK)
- net GPMC0_CSn0: no longer names the net of U23.R19 (GPMC0_CSN0)
- net GPMC0_CSn1: no longer names the net of U23.R20 (GPMC0_CSN1)
- net GPMC0_CSn2: no longer names the net of U23.P19 (GPMC0_CSN2)
- net GPMC0_CSn3: no longer names the net of U23.R21 (GPMC0_CSN3)
- net GPMC0_DIR: no longer names the net of U23.N17 (GPMC0_DIR)
- net GPMC0_OEn_REn: no longer names the net of U23.R18 (GPMC0_OEN_REN)
- net GPMC0_WAIT0: no longer names the net of U23.W19 (GPMC0_WAIT0)
- net GPMC0_WAIT1: no longer names the net of U23.Y18 (GPMC0_WAIT1)
- net GPMC0_WEn: no longer names the net of U23.T21 (GPMC0_WEN)
- net GPMC0_WPn: no longer names the net of U23.N16 (GPMC0_WPN)
- no-connect marks 2 -> 14
Other:
- note removed: "FSI CONNECTOR"
- note removed: "From IO Expander"
- note removed: "GPMC TO FSI & HSE CONNECTOR"
- note removed: "Off Page Connections"
- note removed: "To FSI Mux & HSE"
- note removed: "To HSE"
- note removed: "To HSE & FSI Mux"
- note removed: "To HSE CON"
- note removed: "To HSE Connector"
- note removed: "To MIPI Connector"
