File: 29.kicad_sch (KiCad schematic)
At the start: 75 parts, among them J10 HDR_1X2, J12 HDR_2X1, J31 HDR_1X3, J32 HDR_1X3, J36 CON_FLEX_1X14_10051922, J9 HDR_1X2, U23 AM6442BSFGHAALV, U3 TCAN1042HGVD, U4 TCAN1042HGVD, U67 SN74CB3Q3257PWR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

Commit message: fix joint, offpage, and typo
DRC errors are cleared, some warnings remain.
Parts:
- removed *: TI_TITLEBLK_CSIZE, symbol 29-altium-import:root_0_TI_TITLEBLK_CSIZE
Connections:
- net DGND: now also R541.1
- net MCAN0_H: now also R4.1
- net MCAN0_L: now also R5.2
- net MCAN0_RX: now also J9.1
- net MCAN0_STB_3V3: now also R9.2
- net MCAN0_TX: now also J9.2
- net MCAN1_H: now also R2.1
- net MCAN1_L: now also R3.2
- net MCAN1_RX: now also J10.1
- net MCAN1_STB_3V3: now also R8.2
- net MCAN1_T: now also R2.2, R3.1
- net MCAN1_TX: now also J10.2
- net SoC_I2C0_SCL_RC: now also C492.1
- net SoC_I2C0_SDA_RC: now also C493.1
- net VCC_3V3_SYS: now also C207.2, C410.2, R353.1, R354.1, R357.1, R394.2, R395.2
- net VCC_CAN: now also C23.2, C24.2
- net VCC_LCD: now also C474.1
- net VDDB_3V3_DISPLAY: now also C455.1, J36.10
- net VDD_2V8: now also J36.7
- net VIO_CAN: now also C3.1, C8.1
- no-connect marks 4 -> 3

Commit message: a lot, mpu power almost ready.
Parts:
- removed ACC9: OSD9616P1673-30, NA, symbol 29-altium-import:root_0_ACCESSORY
- removed C454, C460, C462, C463, C470: 1uF, CAP0402_0-75, symbol 29-altium-import:root_2_CAP_Dup3
- removed C455: 0.1uF, CAP0402_0-75, symbol 29-altium-import:root_1_CAP_Dup3
- removed C473: 4.7uF, CAP0603_1, symbol 29-altium-import:root_0_CAP_Dup1
- removed C474: 2.2uF, CAP0603_1, symbol 29-altium-import:root_0_CAP_Dup1
- removed J36: CON_FLEX_1X14_10051922, CON_FLEX1X14_10051922_S_R_S, symbol 29-altium-import:root_2_mirrored_CON_FLEX_14X1_FH19
- removed R516: 100K, RES0402_0-5, symbol 29-altium-import:root_3_RESISTOR_Dup6
- removed R531: 10K, RES0402_0-5, symbol 29-altium-import:root_2_RESISTOR_Dup6
- removed R538: 4.7K, RES0402_0-5, symbol 29-altium-import:root_0_RESISTOR_Dup4
- removed R541: 820K_1%, RES0402_0-5, symbol 29-altium-import:root_1_RESISTOR_Dup1
- removed TP100, TP30, TP65, TP66, TP71, TP73, TP75: TP20_SMD, TP20_SMD, symbol 29-altium-import:root_0_TESTPOINT
- removed TP13, TP57, TP74: TP20_SMD, TP20_SMD, symbol 29-altium-import:root_2_mirrored_TESTPOINT
- removed U99: TPS22945DCKR, SC70-5_1-1, symbol 29-altium-import:root_0_TPS22945DCKR_SC70-5
Connections:
- net HSE_MCAN0_RX/UART4_TXD: no longer U67.3 (1B2)
- net HSE_MCAN0_TX/UART4_RXD: no longer U67.6 (2B2)
- net HSE_MCAN1_RX/I2C3_SDA: no longer U67.10 (3B2)
- net HSE_MCAN1_TX/I2C3_SCL: no longer U67.13 (4B2)
- net RSVD0: no longer names the net of U23.H16 (RSVD0)
- net RSVD1: no longer names the net of U23.D21 (RSVD1)
- net RSVD2: no longer names the net of U23.G13 (RSVD2)
- net RSVD3: no longer names the net of U23.F17 (RSVD3)
- net RSVD4: no longer names the net of U23.W15 (RSVD4)
- net RSVD5: no longer names the net of U23.V16 (RSVD5)
- net RSVD6: no longer names the net of U23.K2 (RSVD6)
- net RSVD7: no longer names the net of U23.K1 (RSVD7)
- net RSVD8: no longer names the net of U23.F12 (RSVD8)
- no-connect marks 3 -> 15
Other:
- note removed: "16V CAP"
- note removed: "DISPLAY"
- note removed: "DISPLAY CONNECTOR"
