File: 30.kicad_sch (KiCad schematic)
At the start: 45 parts, among them J27 CON_MINIPCI_2X32, J34 HDR_1X3, J35 HDR_1X3, U23 AM6442BSFGHAALV, U88 SN74LVC1G08DBVRE4

Commit message: fix joint, offpage, and typo
DRC errors are cleared, some warnings remain.
Parts:
- removed *: MISTRAL_TITLEBLK_CSIZE, symbol 30-altium-import:root_0_MISTRAL_TITLEBLK_CSIZE
Connections:
- net DGND: now also C431.2, C435.2, C448.2, C449.2, C450.2, J27.A12 (GND), J27.A18 (GND), J27.A20 (GND), J27.A23 (GND), J27.A24 (GND), J27.A27 (GND), J27.A28 (GND), J27.A31 (GND), J27.B13 (GND), J27.B18 (GND), J27.B21 (GND), J27.B22 (GND), J27.B25 (GND), J27.B26 (GND), J27.B29 (GND), J27.B32 (GND), J27.B7 (GND), R333.2, R623.1
- net GPIO_PCIe_RST_OUT: now also R424.2
- net PCIE_SERDES_REFCLK0_N: now also R667.2
- net PCIE_SERDES_REFCLK0_P: now also R668.2
- net SERDES_REFCLK0_N: now also R624.2
- net SERDES_REFCLK0_N_C: now also R333.1, R661.2
- net SERDES_REFCLK0_P: now also R623.2
- net SERDES_REFCLK0_P_C: now also R346.1, R662.2
- net VCC_3V3_SYS: now also C426.1, C435.1, J27.A10 (+3.3V), R482.2, R486.2
- net VMAIN: now also C431.1, C448.1, C449.1, C450.1, J27.A2 (+12V), J27.B1 (+12V), J27.B2 (+12V)
- net at R632.1: now also R624.1, R625.1

Commit message: a lot, mpu power almost ready.
Parts:
- removed R661, R662, R667, R668: 0E, RES0402_0-5, symbol 30-altium-import:root_3_RESISTOR_Dup5
Connections:
- net VMAIN: no longer J27.A2 (+12V), J27.A3 (+12V)
- no-connect marks 16 -> 18
Other:
- note removed: "CLOCK SELECTION"
