File: 31.kicad_sch (KiCad schematic)
At the start: 81 parts, among them U105 CDCI6214RGET, U70 CDCLVC1310RHBR, U71 25MHz, Y4 25.000MHz

Commit message: fix joint, offpage, and typo
DRC errors are cleared, some warnings remain.
Parts:
- removed *: MISTRAL_TITLEBLK_CSIZE, symbol 31-altium-import:root_0_MISTRAL_TITLEBLK_CSIZE
Connections:
- net CDC_OE1/OE4 is gone; now on net CDC_OE1/OE4: R688.2
- net CDC_OE4 is gone; now on net CDC_OE1/OE4: U105.11 (OE/GPIO4)
- net CDCEL_XIN: now also C235.2, R245.1, R255.2
- net CDC_EEPROMSEL: now also R686.2, R687.1
- net CDC_XIN: now also Y4.2
- net CDC_XOUT: now also Y4.1
- net CLKGEN_REFCLK1N: now also R682.1
- net CLKGEN_REFCLK1P: now also R681.1
- net CLKGEN_REFCLK4N: now also R684.1
- net CLKGEN_REFCLK4P: now also R683.1
- net CLKOUT0: now also R257.1, R50.2
- net DGND: now also C225.1, C226.1, C252.1, C34.1, C509.2, C513.2, C517.2, C519.2, C524.2, C525.2, C526.2, C527.2, C533.1, C536.1, C537.1, C538.1, R268.2, R45.2, R53.2, R59.2, R60.2, R61.2, R65.2, R682.2, R684.2, U70.15 (GND), U70.16 (GND), U70.21 (GND), U70.25 (GND), U70.26 (GND), U70.32 (GND), U70.4 (GND), U70.9 (GND)
- net IN_SEL0: now also R248.2, R40.2
- net IN_SEL1: now also R253.1, R45.1
- net PRI_INN: now also C252.2, R262.2, R55.1
- net VCC3V3_REF: now also C509.1, C521.1, C524.1
- net VCC3V3_VCO: now also C513.1, C520.1, C527.1
- net VDD1V8_CLKBUF: now also C536.2, C537.2, C538.2, FB25.2, U70.23 (VDDO), U70.6 (VDDO)
- net VDD3V3_CLKBUF: now also C225.2, C226.2, C234.1, C34.2, FB12.2, R253.2
- net VDDO12: now also C519.1, C523.1, FL17.3 (OUT)
- net VDDO34: now also C517.1, C522.1, FL18.3 (OUT)
- net at R272.1, U70.17 (Y5): now also C262.1, R65.1
- net at C255.1, U70.18 (Y6): now also R61.1
- net at C256.1, U70.20 (Y7): now also R60.1
- net at C257.1, U70.22 (Y8): now also R59.1
- net at C247.1, U70.24 (Y9): now also R53.1
- net CDC_OE1/OE4: now reaches R672.2

Commit message: a lot, mpu power almost ready.
Parts:
- removed C509, C513, C517, C519: 0.47uF, CAP0402_0-75, symbol 31-altium-import:root_0_CAP_Dup3
- removed C520, C521, C522, C523: 4.7uF, CAP0402_0-75, symbol 31-altium-import:root_0_CAP_Dup3
- removed C524, C525, C526, C527: 0.1uF, CAP0402_0-75, symbol 31-altium-import:root_0_CAP_Dup3
- removed C532, C533: 27pF, CAP0402_0-75, symbol 31-altium-import:root_1_CAP_Dup3
- removed FL17, FL18, FL19, FL20: 0.47uF, EMIFIL_NFM21P_0805, symbol 31-altium-import:root_0_CAP_FILTER
- removed R235, R236, R237, R238: 22E_1%, RES0402_0-5, symbol 31-altium-import:root_1_RESISTOR_Dup5
- removed R652, R653, R654, R655: 33E_1%, RES0402_0-5, symbol 31-altium-import:root_1_RESISTOR_Dup6
- removed R656, R672, R686, R687: 4.7K, RES0402_0-5, symbol 31-altium-import:root_0_RESISTOR_Dup4
- removed R659, R660: 0E, RES0402_0-5, symbol 31-altium-import:root_1_RESISTOR_Dup5
- removed R681, R682, R683, R684: 49.9E_1%, RES0402_0-5, symbol 31-altium-import:root_0_RESISTOR
- removed R688: 0E, RES0402_0-5, symbol 31-altium-import:root_3_RESISTOR_Dup5
- removed TP102: TP40_SMD, TP40_SMD, symbol 31-altium-import:root_0_mirrored_TESTPOINT
- removed U105: CDCI6214RGET, QFN24_19-68_160X160_1, symbol 31-altium-import:root_0_CDCI6214RGET_VQFN24
- removed Y4: 25.000MHz, XTAL_ABM3_205X130_SMD_1-4, symbol 31-altium-import:root_1_CRY
Connections:
- no-connect marks 8 -> 6
Other:
- note removed: "100MHz HCSL CLK for SoC"
- note removed: "100MHz HCSL CLK to PCIe CON J27"
- note removed: "From GPIO Expander"
- note removed: "PCIe Clock HCSL (100MHz)"
- note removed: "REFSEL-0 selects crystal reference"
