File: 32.kicad_sch (KiCad schematic)
At the start: 26 parts, among them J3 HDR_2X10, U23 AM6442BSFGHAALV, U34 TPIC2810D

Commit message: fix joint, offpage, and typo
DRC errors are cleared, some warnings remain.
Parts:
- removed *: MISTRAL_TITLEBLK_CSIZE, symbol 32-altium-import:root_0_MISTRAL_TITLEBLK_CSIZE
Connections:
- net DGND: now also J3.12, J3.20, J3.5, J3.9, R402.1, R413.1, U34.8 (~{G})
- net VCC_3V3_SYS: now also C147.1, R381.1, R382.1, R383.1, R418.1, R419.1, R420.1, R421.1
- net VDDA_ADC: now also C4.2, C7.2

Commit message: a lot, mpu power almost ready.
Parts:
- removed C147: 0.1uF, CAP0402_0-75, symbol 32-altium-import:root_1_CAP_Dup3
- removed C4, C7: 0.1uF, CAP0402_0-75, symbol 32-altium-import:root_2_CAP_Dup3
- removed J3: HDR_2X10, HDR_2X10_TSW_100_S_T, symbol 32-altium-import:root_0_HEADER_10X2
- removed LD11, LD12, LD13, LD14, LD17, LD18, LD19: 150080VS75000, LED_150080VS75000_80X50_SMD_0-8, symbol 32-altium-import:root_3_mirrored_DIODE_LED
- removed LD16: 150080VS75000, LED_150080VS75000_80X50_SMD_0-8, symbol 32-altium-import:root_3_DIODE_LED
- removed R381, R382, R383, R384, R418, R419, R420, R421: 220E, RES0402_0-5, symbol 32-altium-import:root_0_RESISTOR_Dup6
- removed R401, R402, R413: 10K, RES0402_0-5, symbol 32-altium-import:root_2_RESISTOR_Dup6
- removed U34: TPIC2810D, SOIC16_1-8, symbol 32-altium-import:root_0_TPIC2810D_SOIC16
Connections:
- no-connect marks 2 -> 0
Other:
- note removed: "ETHERNET LED's"
