File: 33.kicad_sch (KiCad schematic)
At the start: 17 parts, among them J5 HDR_1X3, U10 TXS0102DCUR, U91 TCA6424ARGJR

Commit message: fix joint, offpage, and typo
DRC errors are cleared, some warnings remain.
Parts:
- removed *: MISTRAL_TITLEBLK_CSIZE, symbol 33-altium-import:root_0_MISTRAL_TITLEBLK_CSIZE
Connections:
- net DGND: now also U91.25 (GND), U91.33 (EP)
- net VCC1V8: now also C30.2
- net VCC_3V3_SYS: now also C22.2, C444.2, U91.27 (VCCP), U91.31 (VCC)

Commit message: a lot, mpu power almost ready.
Parts:
- removed J5: HDR_1X3, HDR_3X1_100_S_T, symbol 33-altium-import:root_2_HEADER_3X1
Connections:
- net CDC_OE1/OE4: no longer names the net of U91.18 (P21)
- net CPSW_FET_SEL: no longer names the net of U91.11 (P12)
- net FSI_FET_SEL: no longer names the net of U91.8 (P07)
- net GPIO_OLED_RESETn: no longer names the net of U91.15 (P16)
- net GPIO_RGMII1_RST: no longer names the net of U91.4 (P03)
- net GPIO_RGMII2_RST: no longer names the net of U91.5 (P04)
- net PRG1_RGMII2_FET_SEL: no longer names the net of U91.13 (P14)
- net TEST_GPIO2: no longer names the net of U91.14 (P15)
- no-connect marks 0 -> 8
Other:
- note removed: "3V3 IO level"
- note removed: "GND"
- note removed: "I2C TEST HEADER"
- note removed: "SCL"
- note removed: "SDA"
