File: 34.kicad_sch (KiCad schematic)
At the start: 44 parts, among them J1 HDR_2X12, Q8 IRLML6401, SW6 SKHMQLE010, U23 AM6442BSFGHAALV, U35 SN74LVC1G11DCKR, Y1 25.000MHz

Commit message: fix joint, offpage, and typo
DRC errors are cleared, some warnings remain.
Parts:
- removed *: MISTRAL_TITLEBLK_CSIZE, symbol 34-altium-import:root_0_MISTRAL_TITLEBLK_CSIZE
Connections:
- net DGND: now also C134.1, C466.1, C5.1, D9.1, SW6.4, SW6.5 (GND), Y1.4 (GND2)
- net Debounce_MCU_RESETz: now also C466.2, D9.2, R536.1
- net MCU_I2C0_SCL_RC: now also C487.1
- net MCU_I2C0_SDA_RC: now also C488.1
- net MCU_OSC0_XI: now also R137.2
- net MCU_OSC0_XO: now also R140.2
- net MCU_PORz: now also R575.2
- net PORz: now also R574.2
- net PRG1_RGMII_INTn_RC: now also C491.1
- net SoC_WARM_RESETZ: now also TP70.1 (TP)
- net VCC1V8: now also C485.2
- net VCC_3V3_SYS: now also C5.2, R303.1, R309.1
- net at Y1.1: now also C133.2, R138.1
- net at Y1.3: now also C134.2, R139.1
