File: 35.kicad_sch (KiCad schematic)
At the start: 42 parts, among them Q10 IRLML6401, Q17 IRLML6401, Q9 IRLML6401, SW4 SKHMQLE010, SW5 SKHMQLE010, SW7 SKHMQLE010, U41 SN74LVC1G11DCKR, U50 SN74LVC3G17DCUR, U57 SN74LVC1G17DCKR, U74 TPS3711DDCR, U76 TPS3897ADRYR

Commit message: fix joint, offpage, and typo
DRC errors are cleared, some warnings remain.
Parts:
- removed *: MISTRAL_TITLEBLK_CSIZE, symbol 35-altium-import:root_0_MISTRAL_TITLEBLK_CSIZE
Connections:
- net DGND: now also C465.1, C467.1, C468.1, D10.1, D11.1, D8.1, R260.2, SW4.4, SW4.5 (GND), SW5.4, SW5.5 (GND), SW7.4, SW7.5 (GND), U57.3 (GND), U74.2 (GND), U74.4 (GND)
- net Debounce_GPIO_SoC/MCU: now also C465.2, D8.2, R534.1
- net Debounce_WARM_RST: now also C467.2, D11.2, R537.1
- net GPIO_SoC/MCU: now also R470.1, R471.1
- net PORz: now also TP32.1 (TP)
- net SOC_POWER_MON_PORz: now also R285.2
- net SUPERVISOR_DEBOUNCE_RSTn: now also C468.2, D10.2, R540.1
- net SoC_WARM_RESETZ: now also R476.1
- net VCC3V3_PREREG: now also C179.2, C283.2
- net VCC_3V3_SYS: now also C151.2, C173.2
- net VCC_5V0: now also C271.2
- net VDDAR_SENSE: now also R284.2
- net VIN_MON_PORz_3V3_PG: now also C57.1, R259.2
- net at C245.1: now also R260.1, R266.2, U74.3 (SENSE)
Other:
- moved on the sheet: D8

Commit message: a lot, mpu power almost ready.
Parts:
- removed Q10, Q17, Q9: IRLML6401, TO_SOT23-123, symbol 35-altium-import:root_0_MOSFET_IRLML6401TR
- removed R282: 6.34K_1%, RES0402_0-5, symbol 35-altium-import:root_0_RESISTOR
Other:
- note removed: "R2"
