File: 36.kicad_sch (KiCad schematic)
At the start: 44 parts, among them J6 CON_PWRJACK2_PJ-080BH, Q1 BSS138LT1G, Q11 BSS138LT1G, Q2 BSS138LT1G, Q5 BSS138LT1G, Q6 BSS138LT1G, Q7 BSS138LT1G

Commit message: fix joint, offpage, and typo
DRC errors are cleared, some warnings remain.
Parts:
- removed *: MISTRAL_TITLEBLK_CSIZE, symbol 36-altium-import:root_0_MISTRAL_TITLEBLK_CSIZE
Connections:
- net DGND: now also R566.2
- net SHIELD: now also J6.SH1, J6.SH3, R566.1
- net VMAIN: now also C56.1, D3.3 (K)
- net at D1.1 (CATHODE): now also D3.1 (A1), D3.2 (A2), F1.2, R64.1

Commit message: a lot, mpu power almost ready.
Parts:
- removed C478: 1000pF, CAP1206_1-75, symbol 36-altium-import:root_1_CAP_Dup3
- removed C56: 100uF_50V, CAPAE_D8CASE_8, symbol 36-altium-import:root_0_CAP_POL_Dup1
- removed D1: SMCJ64CA, DIO_SMC, symbol 36-altium-import:root_1_DIODE_TVS_DUAL
- removed D2: S1G-13-F, DIO_SMA, symbol 36-altium-import:root_1_DIODE
- removed D3: PMEG045V150EPDAZ, CFP15_PMEG045V150EPD_0-9, symbol 36-altium-import:root_0_DIODE_SCHOTTKY_POWERMITE-3
- removed F1: 10A, FUSE_397_410X110_SMD_2-9, symbol 36-altium-import:root_0_FUSE
- removed J6: CON_PWRJACK2_PJ-080BH, CON_PWRJACK2_PJ-080BH_P_R_T_13-4, symbol 36-altium-import:root_0_mirrored_CON_PWRJACK2_PJ-082BH
- removed LD10, LD2, LD3, LD6, LD7, LD8: 150080VS75000, LED_150080VS75000_80X50_SMD_0-8, symbol 36-altium-import:root_3_mirrored_DIODE_LED
- removed LD5: 150080RS75000, LED_150080VS75000_80X50_SMD_0-8, symbol 36-altium-import:root_1_mirrored_DIODE_LED
- removed Q1, Q2, Q5, Q6, Q7: BSS138LT1G, SOT23-123_1-2, symbol 36-altium-import:root_0_MOSFET_BSS138LT1G
- removed R127, R136, R14, R20, R312: 0E, RES0402_0-5, symbol 36-altium-import:root_3_RESISTOR_Dup5
- removed R15, R211, R305, R360, R365: 220E, RES0402_0-5, symbol 36-altium-import:root_2_RESISTOR_Dup6
- removed R566: 1M, RES0603_0-75, symbol 36-altium-import:root_1_RESISTOR_Dup6
- removed R64: 10K, RES1206_0-75, symbol 36-altium-import:root_0_RESISTOR_Dup1
- removed R80: 1K_1%, RES0402_0-5, symbol 36-altium-import:root_2_RESISTOR_Dup5
- removed TP81: THRU HOLE, TP_40X65, symbol 36-altium-import:root_0_mirrored_TESTPOINT
Other:
- note removed: "Condition"
- note removed: "LED Status(LD1)"
- note removed: "ON"
- note removed: "RED"
- note removed: "Reverse Voltage"
