File: 37.kicad_sch (KiCad schematic)
At the start: 87 parts, among them SW1 ATE1D-6M3-10-Z, U102 SN74LVC1G32DBVR, U17 TPS54334DRCT, U21 CSD18543Q3A, U22 CSD18543Q3A, U24 CSD18543Q3A, U26 CSD18543Q3A, U30 LM5140QRWGTQ1

Commit message: fix joint, offpage, and typo
DRC errors are cleared, some warnings remain.
Parts:
- removed *: MISTRAL_TITLEBLK_CSIZE, symbol 37-altium-import:root_0_MISTRAL_TITLEBLK_CSIZE
Connections:
- net DGND: now also C107.2, C125.2, C135.1, C40.2, C49.2, C65.1, R694.2, SW1.1, SW1.SH1, U17.11 (EP), U17.4 (GND), U17.5 (GND), U21.1 (S1), U21.2 (S2), U22.1 (S1), U22.2 (S2), U30.14 (PGND2), U30.35 (AGND), U30.38 (SYNIN), U30.41 (EP)
- net LM5140_COMP1: now also C135.2
- net LM5140_COMP2: now also C130.1
- net VCC3V3_PREREG: now also C40.1, C46.1, L3.2, R277.1, TP12.1 (TP)
- net VCC3V3_SYS_PG: now also C118.1, R131.2
- net VCC3V3_TA: now also C494.2
- net VCC_3V3_SYS: now also C70.1, C84.1, R113.1, TP44.1 (TP)
- net VCC_5V0: now also C539.1, C69.1, C71.1, R109.1, TP18.1 (TP)
- net VCC_LM5140: now also C107.1, D4.2 (ANODE), D5.2 (ANODE), U30.15 (VCC)
- net VDDA_LM5140: now also R693.1, R701.1
- net VMAIN: now also C123.1, C65.2, C81.1, U17.1 (VIN), U24.5 (D), U26.5 (D)
- net VMAIN_EN: now also C406.1, R408.1, SW1.2
- net VSENSE: now also C272.2, R279.2, R294.1
- net at L3.1, U17.2 (SW): now also C54.1
- net at U24.1 (S1): now also C115.2, L6.2, U21.5 (D), U24.2 (S2), U24.3 (S3), U30.21 (SW1)
- net at R130.1, U24.4 (G): now also U30.23 (HOL1)
- net at R317.2, U22.4 (G): now also R321.2
- net at U22.5 (D): now also C116.1, L5.1, U26.1 (S1), U26.2 (S2), U26.3 (S3), U30.10 (SW2)
- net at R579.1, U17.8 (EN): now also R602.2
- net at R82.1: now also C49.1, U17.7 (COMP)
- net at R319.1: now also R318.1, U21.4 (G)
- net at R129.2, U26.4 (G): now also U30.8 (HOL2)
- net at C272.1: now also R277.2, R279.1
- net at L6.1, R116.2: now also R119.1
- net at C85.1: now also R112.2, U30.4 (CS2)
- net at C85.2: now also R109.2, U30.5 (VOUT2)
- net at C115.1, U30.20 (HB1): now also D4.1 (CATHODE)
- net at C116.2, U30.11 (HB2): now also D5.1 (CATHODE)
- net at R113.2, U30.26 (VOUT1): now also C94.1
- net at R119.2, U30.27 (CS1): now also C94.2
- net at L5.2, R111.1: now also R112.1
Other:
- moved on the sheet: L3, R694, U24, U26

Commit message: a lot, mpu power almost ready.
Parts:
- removed C107, C108: 2.2uF, CAP0603_1, symbol 37-altium-import:root_0_CAP
- removed C115, C116, C494, C54: 0.1uF, CAP0402_0-75, symbol 37-altium-import:root_3_CAP_Dup3
- removed C118, C136, C406: 0.01uF, CAP0402N, symbol 37-altium-import:root_0_CAP_Dup2
- removed C123, C69, C81, C82: 47uF, CAP1206_2, symbol 37-altium-import:root_0_CAP
- removed C125: 3900pF, CAP0402_0-75, symbol 37-altium-import:root_0_CAP_Dup3
- removed C130: 4.7pF, CAP0402N, symbol 37-altium-import:root_0_CAP_Dup2
- removed C131, C132: 0.056uF, CAP0402_0-75, symbol 37-altium-import:root_0_CAP_Dup3
- removed C135: 33pF, CAP0402_0-75, symbol 37-altium-import:root_2_CAP
- removed C137: 1uF, CAP0402_0-75, symbol 37-altium-import:root_2_CAP_Dup3
- removed C138: 0.47uF, CAP0603_1, symbol 37-altium-import:root_0_CAP
- removed C272: 200pF, CAP0402_0-75, symbol 37-altium-import:root_0_CAP_Dup3
- removed C40, C46: 22uF, CAP0603_1, symbol 37-altium-import:root_0_CAP_Dup3
- removed C48: 0.015uF, CAP0402_0-75, symbol 37-altium-import:root_2_CAP_Dup3
- removed C49: 150pF, CAP0402_0-75, symbol 37-altium-import:root_0_CAP_Dup3
- removed C539: 2.2uF, CAP0603_1, symbol 37-altium-import:root_1_CAP
- removed C65: 0.1uF, CAP0402_0-75, symbol 37-altium-import:root_2_CAP_Dup3
- removed C66: 10uF, CAP0603_1, symbol 37-altium-import:root_0_CAP_Dup3
- removed C70: 470uF_10V, CAPAE_875115252003_330X330_SMD_8-7, symbol 37-altium-import:root_0_CAP_POL
- removed C71: 47uF, CAP1206_2, symbol 37-altium-import:root_0_CAP_Dup3
- removed C84: 22uF, CAP1206_2, symbol 37-altium-import:root_0_CAP_Dup3
- removed C85, C94: 33pF, CAP0402_0-75, symbol 37-altium-import:root_1_CAP
- removed D4, D5: XBS104S13R, DIO_SOD323_1, symbol 37-altium-import:root_3_mirrored_DIODE_SCHOTTKY
- removed L3: 6.8uH, IND_74439346068_260X270_SMD_6-1, symbol 37-altium-import:root_1_INDUCTOR_Dup1
- removed L5: 5.6uH, IND_744316100_230X220_SMD_4-3, symbol 37-altium-import:root_1_INDUCTOR_Dup1
- removed L6: 1.5uH, IND_74437349012_270X270_SMD_5, symbol 37-altium-import:root_1_INDUCTOR
- removed R109, R113: 0E, RES0402_0-5, symbol 37-altium-import:root_0_RESISTOR_Dup1
- removed R111: 0.015E_1%, RES1206_1, symbol 37-altium-import:root_1_RESISTOR_Dup1
- removed R112, R119: 49.9E_1%, RES0402_0-5, symbol 37-altium-import:root_0_RESISTOR
- removed R116: 0.006E_1%, RES1206_0-75, symbol 37-altium-import:root_1_RESISTOR_Dup6
- removed R129, R130, R317, R318, R319, R321: 10.2E_1%, RES0402_0-5, symbol 37-altium-import:root_1_RESISTOR_Dup6
- removed R131: 10K_1%, RES0402_0-5, symbol 37-altium-import:root_0_RESISTOR_Dup5
- removed R134, R408: 100K, RES0402_0-5, symbol 37-altium-import:root_2_RESISTOR_Dup6
- removed R141: 3.92K_1%, RES0402_0-5, symbol 37-altium-import:root_1_RESISTOR_Dup6
- removed R142: 2.2K, RES0402_0-5, symbol 37-altium-import:root_3_RESISTOR_Dup6
- removed R277: 51.1E_1%, RES0402_0-5, symbol 37-altium-import:root_0_RESISTOR_Dup6
- removed R279: 31.6K_1%, RES0402_0-5, symbol 37-altium-import:root_0_RESISTOR_Dup6
- removed R294: 10K_1%, RES0402_0-5, symbol 37-altium-import:root_0_RESISTOR_Dup6
- removed R412, R577, R578, R579: 0E, RES0402_0-5, symbol 37-altium-import:root_3_RESISTOR_Dup5
- removed R602: 10K, RES0402_0-5, symbol 37-altium-import:root_2_RESISTOR_Dup6
- removed R693, R694, R700, R701: 0E, RES0402_0-5, symbol 37-altium-import:root_0_RESISTOR_Dup5
- removed R695: 2.2E, RES0603_0-75, symbol 37-altium-import:root_0_RESISTOR_Dup6
- removed R82: 2.05K_1%, RES0402_0-5, symbol 37-altium-import:root_0_RESISTOR_Dup6
- removed SW1: ATE1D-6M3-10-Z, SW3_ATE1F-6M3_370X710_TH_5-6, symbol 37-altium-import:root_0_SW3_B12JV
- removed TP12, TP18, TP44: THRU HOLE, TP_40X65, symbol 37-altium-import:root_0_mirrored_TESTPOINT
- removed U102: SN74LVC1G32DBVR, SOT23-5_1-5, symbol 37-altium-import:root_0_SN74LVC1G32DBVR_SOT23-5
- removed U17: TPS54334DRCT, SON10_19-68_125X125_1, symbol 37-altium-import:root_0_TPS54334DRCT_VSON10
- removed U21: CSD18543Q3A, VSONP8_CSD18543Q_120X130_0-9, symbol 37-altium-import:root_2_MOSFET_CSD18501Q5A
- removed U22: CSD18543Q3A, VSONP8_CSD18543Q_120X130_0-9, symbol 37-altium-import:root_2_mirrored_MOSFET_CSD18501Q5A
- removed U24: CSD18543Q3A, VSONP8_CSD18543Q_120X130_0-9, symbol 37-altium-import:root_0_MOSFET_CSD18501Q5A
- removed U26: CSD18543Q3A, VSONP8_CSD18543Q_120X130_0-9, symbol 37-altium-import:root_0_mirrored_MOSFET_CSD18501Q5A
- removed U30: LM5140QRWGTQ1, TBD, symbol 37-altium-import:root_0_LM5140QRWGTQ1_VQFNP40
- added C118: 10n,50V, Abacus:C_0603_1608Metric_1.28x0.64mm_Courtyard, symbol JLC_C0603:10n,±10%,50V
- added C12, C272: 100p,5%,50V, Abacus:C_0603_1608Metric_1.28x0.64mm_Courtyard, symbol JLC_C0603:100p,5%,50V
- added C123, C66: 4.7u,10%,25V, Capacitor_SMD:C_0805_2012Metric, symbol JLC_C0805:4.7u,10%,25V
- added C13, C14, C15, C46, C48, C49: 22u,20%,25V, Capacitor_SMD:C_0805_2012Metric, symbol JLC_C0805:22u,20%,25V
- added L3, L6: 470nH,15mOhm, Inductor_SMD:L_Sunlord_MWSA0518S, symbol Device:L
- added R12, R279: 68k,1%, Abacus:R_0603_1608Metric_1.28x0.64mm_Courtyard, symbol JLC_R0603:68k,1%
- added R131: 10k,1%, Abacus:R_0603_1608Metric_1.28x0.64mm_Courtyard, symbol JLC_R0603:10k,1%
- added R21, R294: 15k,1%, Abacus:R_0603_1608Metric_1.28x0.64mm_Courtyard, symbol JLC_R0603:15k,1%
- added R22: 0R,1%, Abacus:R_0402_1005Metric_for_0.25mm_grid, symbol JLC_R0402:0R,1%
- added TP8: THRU HOLE, TP_40X65, symbol 37-altium-import:root_0_mirrored_TESTPOINT
- added U17, U30: TPS62826, Abacus:Texas_VSON-HR-6_1.5x1.5mm_P0.5mm, symbol Abacus:TPS62826
Connections:
- net VCC3V3_PREREG: now also C272.1, C46.1, C48.1, C49.1, L3.2, R279.1
- net VCC3V3_SYS_PG: now also C118.1, R131.2, U30.2 (PG)
- net VCC_3V3_SYS: now also C12.1, C13.1, C14.1, C15.1, L6.2, R12.1, R131.1, TP8.1 (TP)
- net VIN_MON_PORz_3V3_PG: now also R22.1, U17.2 (PG)
- new net: L6.1, U30.5 (SW)
- new net: L3.1, U17.5 (SW)
- new net: C272.2, R279.2, R294.1, U17.3 (FB)
- new net: R22.2, U30.1 (EN)
- new net: C12.2, R12.2, R21.1, U30.3 (FB)
- new net +5V: C123.1, C66.1, U17.1 (EN), U17.6 (VIN), U30.6 (VIN)
- new net GND: C118.2, C123.2, C13.2, C14.2, C15.2, C46.2, C48.2, C49.2, C66.2, R21.2, R294.2, U17.4 (GND), U30.4 (GND)
- no-connect marks 3 -> 0
Other:
- note added: "C272 120p preferred"
- note added: "MWSA0518S-R47MT"
- note added: "VIN_MON_PORz_3V3_PG is pulled up in RESET circuitry."
- note removed: "5V,3A and 3.3V,7A Dual SUPPLY"
- note removed: "ON/ OFF Control SWITCH"
- note removed: "VCC3V3_SYS & VCC_5V0 POWER SUPPLY"
