File: 38.kicad_sch (KiCad schematic)
At the start: 64 parts, among them U103 SN74LVC1G32DBVR, U104 SN74LVC1G08DBVRE4, U12 TPS82084SILT, U25 TPS62823DLCT, U33 TPS74601PDRVR, U5 TPS62097RWKT, U65 TPS62087RLTT, U72 TLV75518PDQNR

Commit message: fix joint, offpage, and typo
DRC errors are cleared, some warnings remain.
Parts:
- removed *: MISTRAL_TITLEBLK_CSIZE, symbol 38-altium-import:root_0_MISTRAL_TITLEBLK_CSIZE
Connections:
- net DGND: now also C202.2, U12.5 (GND), U12.9 (EP), U25.3 (AGND), U33.7 (EP), U5.11 (AGND), U72.2 (GND), U72.5 (EP)
- net VCC1V2_DDR: now also C20.1, L2.2, R214.1, TP4.1 (TP), U5.3 (VOS)
- net VCC1V8: now also C217.1, L8.2, TP51.1 (TP), U65.3 (FB), U65.4 (VOS)
- net VCC3V3_PREREG: now also C37.1, C479.1, C495.2, U25.7 (VIN), U33.6 (IN), U5.7 (PVIN), U5.8 (AVIN), U65.7 (VIN), U72.4 (IN)
- net VCC_CORE: now also C486.1, C77.1, L4.2, TP23.1 (TP)
- net VCC_CORE_EN: now also C540.1
- net VCC_CORE_FB: now also C96.2, R117.2, R118.2
- net VDD1V8_PG: now also C403.1, R143.1
- net VDDA1V8: now also C129.1, R144.1
- net VDDAR_CORE: now also R44.1, TP10.1 (TP)
- net VDD_0V85: now also C33.1
- net VDD_CORE: now also R118.1
- net VPP_1V8: now also C243.1, TP52.1 (TP), U72.1 (OUT)
- net VPP_LDO_EN: now also R263.2
- net at R697.1: now also R584.1, U25.1 (EN)
- net at R44.2, R49.1: now also U12.7 (FB)
- net at U5.4 (FB): now also R213.1, R214.2
- net at U33.2 (FB): now also R144.2, R145.1
- no-connect marks 3 -> 2

Commit message: a lot, mpu power almost ready.
Parts:
- removed C126: 1uF, CAP0402_0-75, symbol 38-altium-import:root_0_CAP_Dup3
- removed C129: 2.2uF, CAP0402_0-75, symbol 38-altium-import:root_0_CAP_Dup3
- removed C211: 10uF, CAP0603_1, symbol 38-altium-import:root_0_CAP_Dup3
- removed C217, C33: 22uF, CAP0603_1, symbol 38-altium-import:root_0_CAP_Dup3
- removed C37: 10uF, CAP0402_0-75, symbol 38-altium-import:root_0_CAP_Dup1
- removed C403: 0.01uF, CAP0402N, symbol 38-altium-import:root_0_CAP_Dup2
- removed C479, C540: 0.1uF, CAP0402_0-75, symbol 38-altium-import:root_0_CAP_Dup3
- removed C486, C77: 10uF, CAP0402_0-75, symbol 38-altium-import:root_0_CAP_Dup3
- removed C495: 0.1uF, CAP0402_0-75, symbol 38-altium-import:root_3_CAP_Dup3
- removed C95: 4.7uF, CAP0603_1, symbol 38-altium-import:root_0_CAP_Dup1
- removed C96: 120pF, CAP0402_0-75, symbol 38-altium-import:root_0_CAP
- removed L4, L8: 0.47uH, IND_744373460047_270X270_SMD_3, symbol 38-altium-import:root_1_INDUCTOR
- removed R117, R123, R58: 100K, RES0402_0-5, symbol 38-altium-import:root_2_RESISTOR_Dup6
- removed R118: 24.9K_1%, RES0402_0-5, symbol 38-altium-import:root_0_RESISTOR
- removed R143: 10K, RES0402_0-5, symbol 38-altium-import:root_2_RESISTOR_Dup6
- removed R144: 47.5K_1%, RES0402_0-5, symbol 38-altium-import:root_0_RESISTOR_Dup6
- removed R145: 21K_1%, RES0402_0-5, symbol 38-altium-import:root_0_RESISTOR_Dup6
- removed R44: 10.1K_0.1%, RES0603_0-75, symbol 38-altium-import:root_0_RESISTOR_Dup1
- removed R49: 162K_1%, RES0402_0-5, symbol 38-altium-import:root_0_RESISTOR
- removed R57: 0E, RES0402_0-5, symbol 38-altium-import:root_1_RESISTOR_Dup5
- removed R580, R583, R584, R697: 0E, RES0402_0-5, symbol 38-altium-import:root_3_RESISTOR_Dup5
- removed R696: 1K, RES0402_0-5, symbol 38-altium-import:root_3_RESISTOR_Dup5
- removed TP23, TP8: THRU HOLE, TP_40X65, symbol 38-altium-import:root_0_mirrored_TESTPOINT
- removed TP24, TP49: TP20_SMD, TP20_SMD, symbol 38-altium-import:root_0_TESTPOINT
- removed U103: SN74LVC1G32DBVR, SOT23-5_1-5, symbol 38-altium-import:root_0_SN74LVC1G32DBVR_SOT23-5
- removed U104: SN74LVC1G08DBVRE4, SOT23-5, symbol 38-altium-import:root_0_SN74LVC1G08DBVRE4_SOT23-5
- removed U12: TPS82084SILT, uSIP8_TPS82084_110X120_1-4, symbol 38-altium-import:root_0_TPS82084_USIP8
- removed U25: TPS62823DLCT, VSONHR8_TPS62823_60X80_1, symbol 38-altium-import:root_0_TPS62823_VSONHR8
- removed U33: TPS74601PDRVR, SON6_25-59_85X85_0-8, symbol 38-altium-import:root_0_TPS74501_WSON6
- removed U65: TPS62087RLTT, VSONHR7_TPS62085_80X80_1, symbol 38-altium-import:root_0_TPS62085RLTR_VSONHR7
- added C11, C211, C95: 4.7u,10%,25V, Capacitor_SMD:C_0805_2012Metric, symbol JLC_C0805:4.7u,10%,25V
- added C126: 1u,±10%,25V, Abacus:C_0402_1005Metric_for_0.25mm_grid, symbol JLC_C0402:1u,±10%,25V
- added C129: 2.2u,±20%,6.3V, Abacus:C_0402_1005Metric_for_0.25mm_grid, symbol JLC_C0402:2.2u,±20%,6.3V
- added C16, C29, C96: 100p,5%,50V, Abacus:C_0603_1608Metric_1.28x0.64mm_Courtyard, symbol JLC_C0603:100p,5%,50V
- added C17, C18, C19, C31, C32, C33, C486, C77, C78: 22u,20%,25V, Capacitor_SMD:C_0805_2012Metric, symbol JLC_C0805:22u,20%,25V
- added C21, C26: 10n,50V, Abacus:C_0603_1608Metric_1.28x0.64mm_Courtyard, symbol JLC_C0603:10n,±10%,50V
- added L1, L4, L8: 470nH,15mOhm, Inductor_SMD:L_Sunlord_MWSA0518S, symbol Device:L
- added R117: 120k,1%, Abacus:R_0603_1608Metric_1.28x0.64mm_Courtyard, symbol JLC_R0603:120k,1%
- added R118: 49.9k,1%, Abacus:R_0603_1608Metric_1.28x0.64mm_Courtyard, symbol JLC_R0603:49.9k,1%
- added R123, R144, R145: 100k,1%, Abacus:R_0402_1005Metric_for_0.25mm_grid, symbol JLC_R0402:100k,1%
- added R14, R43: 100k,1%, Abacus:R_0603_1608Metric_1.28x0.64mm_Courtyard, symbol JLC_R0603:100k,1%
- added R146: 22k,1%, Abacus:R_0402_1005Metric_for_0.25mm_grid, symbol JLC_R0402:22k,1%
- added R15, R28: 200k,1%, Abacus:R_0603_1608Metric_1.28x0.64mm_Courtyard, symbol JLC_R0603:200k,1%
- added R20, R580: 100R,1%, Abacus:R_0603_1608Metric_1.28x0.64mm_Courtyard, symbol JLC_R0603:100R,1%
- added R583, R697: 0R,1%, Abacus:R_0603_1608Metric_1.28x0.64mm_Courtyard, symbol JLC_R0603:0R,1%
- added TP12: THRU HOLE, TP_40X65, symbol 38-altium-import:root_0_mirrored_TESTPOINT
- added U2, U25, U6: TPS62826, Abacus:Texas_VSON-HR-6_1.5x1.5mm_P0.5mm, symbol Abacus:TPS62826
- added U33: TLV75901PDRV, Package_SON:WSON-6-1EP_2x2mm_P0.65mm_EP1x1.6mm, symbol Abacus:TLV75901PDRV
- TP10: value THRU HOLE -> TP20_SMD; footprint TP_40X65 -> TP20_SMD; CHKD/DATE MAZHAR/271211 -> SHREESHAIL/171006; CRTD /DATE SHREESHAIL/041005 -> MAZHAR/171006; CUSTOMS_HS_CODE (none) -> NA; CUSTOM_DUTY (none) -> NA; FOOTPRINT PATH (none) -> Y~{:}MIS_DATABAS~{E}Librar~{y}ALTIUM_TOO~{L}PCB_FOOTPRINT~{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; FOOTPRINT REF (none) -> TP20_SMD; LIBRARY PATH (none) -> Y~{:}MIS_DATABAS~{E}Librar~{y}ALTIUM_TOO~{L}SCHEMATICS_PART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; MECHANICAL 3D STEP FILE (none) -> NA; MFR_PART_NUMBER TP_40X65 -> TP20_SMD; MISTRAL PART NO 130009030938 -> NA; PACKAGE THRU-HOLE -> SMD; PCB FOOTPRINT TP_40X65 -> TP20_SMD; PROJECT HSE -> BT MODULE_CSRBC04; ROHS (none) -> NA; TEMPERATURE (none) -> NA; TOLERANCE (none) -> NA; VOLTAGE (none) -> NA; WATTAGE (none) -> NA; WEIGHT (none) -> NA
Connections:
- net VDDAR_CORE is gone; now on net VDD1V8_PG: TP10.1 (TP)
- net VCC1V2_PG: now also R697.1
- net VCC1V8: now also C16.1, C17.1, C18.1, C19.1, C29.1, C31.1, C32.1, C33.1, L1.2, L8.2, R15.1, R28.1, TP12.1 (TP)
- net VCC3V3_PREREG: now also C11.1, C126.1, C211.1, R123.1, U2.6 (VIN), U33.6 (IN), U6.6 (VIN)
- net VCC3V3_SYS_PG: now also R583.2
- net VCC_CORE_FB: now also C96.2, R117.1, R118.2, U25.3 (FB)
- net VCC_CORE_PG: now also R123.2, U25.2 (PG)
- net VDD1V8_PG: now also U2.2 (PG), U6.2 (PG)
- net VDD_CORE: now also C486.1, C77.1, C78.1, C96.1, L4.2, R118.1
- net VCC1V2_DDR renamed VDD_DDR4
- net VDDA1V8 renamed VDDA_1V8
- net VDDA_1V8: now also C129.1, R144.1, R145.1, R20.1, R580.1, U33.1 (OUT)
- new net: C16.2, R14.1, R15.2, U2.3 (FB)
- new net: C29.2, R28.2, R43.1, U6.3 (FB)
- new net: L4.1, U25.5 (SW)
- new net: R583.1, U33.4 (EN)
- new net: L8.1, U2.5 (SW)
- new net: C26.1, R20.2, U6.1 (EN)
- new net: R144.2, R145.2, R146.1, U33.2 (FB)
- new net: R697.2, U25.1 (EN)
- new net: C21.1, R580.2, U2.1 (EN)
- new net: L1.1, U6.5 (SW)
- new net +5V: C95.1, U25.6 (VIN)
- new net GND: C11.2, C126.2, C129.2, C17.2, C18.2, C19.2, C21.2, C211.2, C26.2, C31.2, C32.2, C33.2, C486.2, C77.2, C78.2, C95.2, R117.2, R14.2, R146.2, R43.2, U2.4 (GND), U25.4 (GND), U33.3 (GND), U33.7 (GND), U6.4 (GND)
- no-connect marks 2 -> 1
Other:
- note added: "C96 120p preferred"
- note added: "This chip has no PowerGood output, which is logially ANDed with VCC1V8_PG (from DCDC) for DDR power enable in original design. We change the concurrent VCC1V8 and VDDA_1V8 rampups to sequential one, first VDDA_1V8 then VCC1V8."
- note removed: "0.75V"
- note removed: "0.85 V, 1.5 AMPS SUPPLY"
- note removed: "0.85V"
- note removed: "CORE VOLTAGE"
- note removed: "Ren"
- note removed: "Rfb"
- note removed: "Rfb = 24.9K"
- note removed: "Rfb = 41.2K"
- note removed: "Rfb RES TO BE PLACED"
- moved on the sheet: TP14, TP29, TP50, TP51
