File: 39.kicad_sch (KiCad schematic)
At the start: 60 parts, among them U100 TLV70728PDQNR, U32 TPS62097RWKT, U62 TPS73525DRVR, U68 TPS51206DSQR, U77 TLV70710DQNR, U9 TPS62097RWKT, U97 TPS62177DQCR

Commit message: fix joint, offpage, and typo
DRC errors are cleared, some warnings remain.
Parts:
- removed *: MISTRAL_TITLEBLK_CSIZE, symbol 39-altium-import:root_0_MISTRAL_TITLEBLK_CSIZE
Connections:
- net DDR_VREFCA: now also U68.6 (VTTREF)
- net DDR_VTT_EN_3V3: now also U68.9 (S5)
- net DGND: now also U100.2 (GND), U100.5 (EP), U32.1 (PGND), U62.7 (EP), U68.11 (EP), U68.8 (GND), U77.2 (GND), U77.5 (EP), U9.1 (PGND), U97.11 (EP), U97.5 (FB), U97.6 (AGND)
- net VCC3V3_TA: now also C458.1, R535.2, U97.10 (VOS)
- net VCC_3V3_SYS: now also C127.1, C25.1, U100.4 (IN), U32.7 (PVIN), U32.8 (AVIN), U62.6 (IN), U68.10 (VDD), U68.2 (VLDOIN), U77.4 (IN), U9.7 (PVIN), U9.8 (AVIN)
- net VDDR_VTT: now also C210.2, U68.5 (VTTSNS)
- net VDD_1V0: now also C280.1, TP56.1 (TP), U77.1 (OUT)
- net VDD_1V1: now also C122.1, L7.2, R361.1, TP28.1 (TP), U32.3 (VOS)
- net VDD_2V5: now also C28.1, L1.2, R232.1, TP6.1 (TP), U9.3 (VOS)
- net VDD_2V8: now also C471.1, TP99.1 (TP), U100.1 (OUT)
- net VDD_DDR4: now also U68.1 (VDDQSNS)
- net VMAIN: now also C452.1
- net VPP_DDR_2V5: now also U62.1 (OUT)
- net at R361.2, R364.1: now also U32.4 (FB)
- net at R231.1, R232.2: now also U9.4 (FB)
- net at TP98.1 (TP), U97.7 (PG): now also R535.1

Commit message: a lot, mpu power almost ready.
Parts:
- removed C122: 22uF, CAP0603_1, symbol 39-altium-import:root_0_CAP_Dup3
- removed C127: 10uF, CAP0402_0-75, symbol 39-altium-import:root_0_CAP_Dup3
- removed C215, C402: 0.01uF, CAP0402N, symbol 39-altium-import:root_0_CAP_Dup2
- removed C452: 2.2uF, CAP0603_1, symbol 39-altium-import:root_0_CAP
- removed C458: 22uF, CAP0805_1-5, symbol 39-altium-import:root_0_CAP_Dup3
- removed C459, C471: 1uF, CAP0402_0-75, symbol 39-altium-import:root_0_CAP_Dup3
- removed L1, L7: 1uH, IND_744316100_230X220_SMD_4-3, symbol 39-altium-import:root_1_INDUCTOR
- removed L9: 10uH, IND_74438336100_130X130_SMD_2, symbol 39-altium-import:root_1_INDUCTOR
- removed LD24: 150080VS75000, LED_150080VS75000_80X50_SMD_0-8, symbol 39-altium-import:root_3_mirrored_DIODE_LED
- removed LD25: 150080VS75000, LED_150080VS75000_80X50_SMD_0-8, symbol 39-altium-import:root_3_DIODE_LED
- removed R201: 220E, RES0402_0-5, symbol 39-altium-import:root_0_RESISTOR_Dup6
- removed R225, R396, R535: 100K, RES0402_0-5, symbol 39-altium-import:root_2_RESISTOR_Dup6
- removed R231: 4.7K, RES0402_0-5, symbol 39-altium-import:root_0_RESISTOR_Dup4
- removed R232: 10K_1%, RES0402_0-5, symbol 39-altium-import:root_0_RESISTOR_Dup6
- removed R361: 7.5K_1%, RES0402_0-5, symbol 39-altium-import:root_0_RESISTOR
- removed R364: 21K_1%, RES0402_0-5, symbol 39-altium-import:root_0_RESISTOR_Dup1
- removed R500: 0E, RES0402_0-5, symbol 39-altium-import:root_0_RESISTOR_Dup5
- removed R556: 160E_1%, RES0402_0-5, symbol 39-altium-import:root_0_RESISTOR_Dup6
- removed R587, R589: 0E, RES0402_0-5, symbol 39-altium-import:root_3_RESISTOR_Dup5
- removed TP28, TP99: THRU HOLE, TP_40X65, symbol 39-altium-import:root_0_mirrored_TESTPOINT
- removed TP96, TP98: TP20_SMD, TP20_SMD, symbol 39-altium-import:root_0_mirrored_TESTPOINT
- removed TP97: TP20_SMD, TP20_SMD, symbol 39-altium-import:root_0_TESTPOINT
- removed U100: TLV70728PDQNR, X2SON4_TLV71318P_40X40_0-4, symbol 39-altium-import:root_0_TLV71318PDQNR_X2SON4
- removed U32, U9: TPS62097RWKT, VQFNHR11_TPS62097_80X80_1, symbol 39-altium-import:root_0_TPS62097RWKT_VQFNHR11
- removed U97: TPS62177DQCR, WSON10_19-68_80X120_0-8, symbol 39-altium-import:root_0_TPS62177_WSON10
- added U9: TLV73325PDBV, Package_TO_SOT_SMD:SOT-23-5, symbol Regulator_Linear:TLV73325PDBV
Connections:
- net DGND: now also U9.2 (GND)
- net VCC_3V3_SYS: now also U9.1 (IN)
- net VDD_2V5: now also U9.5 (OUT)
- net at R585.1: now also U9.3 (EN)
- no-connect marks 4 -> 1
Other:
- note removed: "1.1 V ETHERNET PHY (DP83869) POWER SUPPLY"
- note removed: "2.8 V , 0.2 AMP SUPPLY"
